File: AstraController/ASTRA - Copy.kicad_sch (KiCad schematic)
At the start: 100 parts, among them J1 Nema17, J2 Nema17, J3 Conn_01x04, J4 Conn_01x04, J6 USB_A_Stacked, P1 12V-DC, Q1 AO3401A, Q2 2N3904, Q3 2N3904, SW1 TOP, SW2 BOTTOM, SW3 LEFT, SW4 RIGHT, SW5 SELECT, SW6 RETURN, SW7 RESET, U1 MCP23017x-x-ML, U2 USB2512B_M2, U3 CH340C, U4 SPX3819M5-L-3-3, U5 ESP32-WROOM-32UE, U6 AP62300WU, U7 TMC2209-LA, U8 TMC2209-LA, Y1 Crystal

Commit message: frame and pcb ver 5.5
Parts:
- removed C35: 10uF, Capacitor_SMD:C_0402_1005Metric, symbol Device:C
- removed C36: 100nF, Capacitor_SMD:C_0402_1005Metric, symbol Device:C
- removed C37, C38: 22uF, Capacitor_SMD:C_0805_2012Metric, symbol Device:C
- removed J1, J2: Nema17, Connector_JST:JST_XH_B4B-XH-A_1x04_P2.50mm_Vertical, symbol Connector_Generic:Conn_01x04
- removed J3, J4: Conn_01x04, Connector_JST:JST_SH_BM04B-SRSS-TB_1x04-1MP_P1.00mm_Vertical, symbol Connector_Generic:Conn_01x04
- removed L2: L_Ferrite, Inductor_SMD:L_Wuerth_WE-PD-Typ-M-Typ-S, symbol Device:L_Ferrite
- removed R25, R26, R27, R28: 0.15R, Resistor_SMD:R_0402_1005Metric, symbol Device:R
- removed R29: 12kR, Resistor_SMD:R_0402_1005Metric, symbol Device:R
- removed R30: 2.2kR, Resistor_SMD:R_0402_1005Metric, symbol Device:R
- removed U1: MCP23017x-x-ML, Package_DFN_QFN:QFN-28-1EP_6x6mm_P0.65mm_EP4.25x4.25mm, symbol Interface_Expansion:MCP23017x-x-ML
- removed U6: AP62300WU, Package_TO_SOT_SMD:TSOT-23-6, symbol Regulator_Switching:AP62300WU
- added B1: XL4016E1 Buck Converter, ASTRAfootprints:Double 1x02 screw connector, symbol Connector_Generic:Conn_01x04
- added C8: 100nF, Capacitor_SMD:C_0402_1005Metric, symbol Device:C
- added J1, J2: RJ45 (NEMA 17), Connector_RJ:RJ45_Amphenol_54602-x08_Horizontal, symbol Connector:RJ45
- added J3, J4: RJ45 (BNO085), Connector_RJ:RJ45_Amphenol_54602-x08_Horizontal, symbol Connector:RJ45
- added U1: MCP23017x-x-SP, Package_DIP:DIP-28_W7.62mm, symbol Interface_Expansion:MCP23017x-x-SP
- C26, C29: value 100nF -> 22nF
- F1: footprint Fuse:Fuse_2920_7451Metric -> (none)
- P1: footprint Connector_JST:JST_VH_B2P-VH_1x02_P3.96mm_Vertical -> TerminalBlock:TerminalBlock_Xinya_XY308-2.54-2P_1x02_P2.54mm_Horizontal
- R9: value 12kR -> 47kR
- S1: footprint Connector_JST:JST_SH_BM08B-SRSS-TB_1x08-1MP_P1.00mm_Vertical -> ASTRAfootprints:Quadruple 1x02 screw connector
- SW1, SW2, SW3, SW4, SW5, SW6, SW7: footprint Connector_JST:JST_SH_BM02B-SRSS-TB_1x02-1MP_P1.00mm_Vertical -> TerminalBlock:TerminalBlock_Xinya_XY308-2.54-2P_1x02_P2.54mm_Horizontal
Connections:
- net +12V: now also B1.1 (Pin_1); no longer C26.2, C29.2
- net +3.3V: now also J3.4, J4.4, U1.9 (V_{DD})
- net +5V: now also B1.3 (Pin_3)
- net BLUE: now also U1.22 (GPA1)
- net BOTTOM: now also U1.3 (GPB2)
- net DTR: now also C8.1; no longer C7.2, R6.1, SW7.2, U5.3 (EN)
- net GND: now also C26.2, C29.2, U7.23 (BRA), U7.27 (BRB), U8.23 (BRA), U8.27 (BRB), B1.2 (Pin_2), B1.4 (Pin_4), J3.2, J3.5, J3.6, J4.2, J4.5, J4.6, U1.10 (V_{SS}), U1.15 (A0), U1.16 (A1), U1.17 (A2); no longer U7.13 (CLK), U8.13 (CLK)
- net GREEN: now also U1.7 (GPB6)
- net LEFT: now also U1.4 (GPB3)
- net RED: now also U1.6 (GPB5)
- net RETURN: now also U1.1 (GPB0)
- net RIGHT: now also U1.5 (GPB4)
- net SCL: now also J3.3, J4.3, U1.12 (SCK)
- net SDA: now also J3.1, J4.1, U1.13 (SDA)
- net SELECT: now also U1.28 (GPA7)
- net TOP: now also U1.2 (GPB1)
- net WHITE: now also U1.8 (GPB7)
- net YELLOW: now also U1.21 (GPA0)
- net at U7.1 (OB2): now also J1.7, J1.8
- net at U7.21 (OA2): now also J1.3, J1.4
- net at U7.24 (OA1): now also J1.1, J1.2
- net at U7.26 (OB1): now also J1.5, J1.6
- net at U8.24 (OA1): now also J2.1, J2.2
- net at U8.21 (OA2): now also J2.3, J2.4
- net at U8.26 (OB1): now also J2.5, J2.6
- net at U8.1 (OB2): now also J2.7, J2.8
- net at C33.2, R19.1: now also U1.18 (~{RESET})
- new net: C7.2, C8.2, R6.1, SW7.2, U5.3 (EN)
