File: AstraController/ASTRA.kicad_sch (KiCad schematic)
At the start: 100 parts, among them J1 Nema17, J2 Nema17, J3 Conn_01x04, J4 Conn_01x04, J6 USB_A_Stacked, P1 12V-DC, Q1 AO3401A, Q2 2N3904, Q3 2N3904, SW1 TOP, SW2 BOTTOM, SW3 LEFT, SW4 RIGHT, SW5 SELECT, SW6 RETURN, SW7 RESET, U1 MCP23017x-x-ML, U2 USB2512B_M2, U3 CH340C, U4 SPX3819M5-L-3-3, U5 ESP32-WROOM-32UE, U6 AP62300WU, U7 TMC2209-LA, U8 TMC2209-LA, Y1 Crystal

Commit message: temp commit
Parts:
- removed J2: Nema17, Connector_JST:JST_XH_B4B-XH-A_1x04_P2.50mm_Vertical, symbol Connector_Generic:Conn_01x04
- removed R24: 10kR, Resistor_SMD:R_0402_1005Metric, symbol Device:R
- removed Y1: Crystal, Crystal:Crystal_SMD_3225-4Pin_3.2x2.5mm, symbol Device:Crystal
- added D6: D_Zener, symbol Device:D_Zener
- added J2: Nema17, symbol Connector_Generic:Conn_01x06
- added R31: 47kR, Resistor_SMD:R_0402_1005Metric, symbol Device:R
- added R32: 6.8kR, Resistor_SMD:R_0402_1005Metric, symbol Device:R
- added Y1: Crystal_GND24, symbol Device:Crystal_GND24
- C35: footprint Capacitor_SMD:C_0402_1005Metric -> Capacitor_SMD:C_0805_2012Metric
- J1: footprint Connector_JST:JST_XH_B4B-XH-A_1x04_P2.50mm_Vertical -> Connector_JST:JST_PH_B6B-PH-K_1x06_P2.00mm_Vertical
Connections:
- net +12V: now also C35.2, Q1.2 (S), D6.1 (K), R31.1; no longer C35.1, Q1.3 (D), U6.5 (EN)
- net +3.3V: now also C9.1, U3.16 (VCC), U3.4 (V3)
- net +5V: no longer U3.16 (VCC)
- net DTR: now also Q2.1 (E), R22.2, U3.13 (~{DTR}); no longer C7.2, Q3.3 (C), R6.1, SW7.2, U5.3 (EN)
- net GND: now also C35.1, R32.2; no longer C35.2, Q2.1 (E), Q3.1 (E)
- net RTS: now also Q3.1 (E), R23.2, U3.14 (~{RTS}); no longer Q2.3 (C), U5.25 (IO0)
- net at Q1.1 (G), R21.1: now also D6.2 (A)
- net at F1.1: now also Q1.3 (D); no longer Q1.2 (S)
- net at C24.2: now also Y1.1
- net at C23.1: now also Y1.3
- new net: R31.2, R32.1, U6.5 (EN)
- new net: Y1.2 (G), Y1.4 (G)
- new net ESP32EN: C7.2, Q3.3 (C), R6.1, SW7.2, U5.3 (EN)
- new net GPIO0: Q2.3 (C), U5.25 (IO0)
Other:
- moved on the sheet: Q2

Commit message: new schem
Parts:
- removed C1: 680uF, Capacitor_THT:CP_Radial_D10.0mm_P5.00mm, symbol Device:C_Polarized
- removed C10, C11, C12, C13, C14, C16, C17, C19, C2, C21, C22, C26, C29, C3, C32, C36, C4, C6, C9: 100nF, Capacitor_SMD:C_0402_1005Metric, symbol Device:C
- removed C15, C25, C33, C34, C35: 10uF, Capacitor_SMD:C_0805_2012Metric, symbol Device:C
- removed C18, C20: 10nF, Capacitor_SMD:C_0402_1005Metric, symbol Device:C
- removed C23, C24: 18pF, Capacitor_SMD:C_0402_1005Metric, symbol Device:C
- removed C27, C31: 2.2uF, Capacitor_SMD:C_0402_1005Metric, symbol Device:C
- removed C28, C30: 22nF, Capacitor_SMD:C_0402_1005Metric, symbol Device:C
- removed C37, C38: 22uF, Capacitor_SMD:C_0805_2012Metric, symbol Device:C
- removed C7: 1uF, Capacitor_SMD:C_0402_1005Metric, symbol Device:C
- removed D1: LED_RED, LED_SMD:LED_0805_2012Metric, symbol Device:LED
- removed D2: LED_GREEN, LED_SMD:LED_0805_2012Metric, symbol Device:LED
- removed D3: LED_WHITE, LED_SMD:LED_0805_2012Metric, symbol Device:LED
- removed D4: LED_BLUE, LED_SMD:LED_0805_2012Metric, symbol Device:LED
- removed D5: LED_YELLOW, LED_SMD:LED_0805_2012Metric, symbol Device:LED
- removed D6: D_Zener, symbol Device:D_Zener
- removed F1: Polyfuse, Fuse:Fuse_2920_7451Metric, symbol Device:Polyfuse
- removed G1: BNO085, Connector_PinSocket_2.54mm:PinSocket_1x09_P2.54mm_Vertical, symbol Connector_Generic:Conn_01x09
- removed J1: Nema17, Connector_JST:JST_PH_B6B-PH-K_1x06_P2.00mm_Vertical, symbol Connector_Generic:Conn_01x04
- removed J2: Nema17, symbol Connector_Generic:Conn_01x06
- removed J3, J4: Conn_01x04, Connector_JST:JST_SH_BM04B-SRSS-TB_1x04-1MP_P1.00mm_Vertical, symbol Connector_Generic:Conn_01x04
- removed J6: USB_A_Stacked, Connector_USB:USB_A_CUI_UJ2-ADH-TH_Horizontal_Stacked, symbol Connector:USB_A_Stacked
- removed L2: L_Ferrite, Inductor_SMD:L_Wuerth_WE-PD-Typ-M-Typ-S, symbol Device:L_Ferrite
- removed P1: 12V-DC, Connector_JST:JST_VH_B2P-VH_1x02_P3.96mm_Vertical, symbol Connector:Jack-DC
- removed Q1: AO3401A, Package_TO_SOT_SMD:SOT-23, symbol Transistor_FET:AO3401A
- removed Q2, Q3: 2N3904, Package_TO_SOT_THT:TO-92_Inline, symbol Transistor_BJT:2N3904
- removed R1, R2, R3, R4, R5: 100R, Resistor_SMD:R_0402_1005Metric, symbol Device:R
- removed R10, R19, R20, R21, R22, R23, R6: 10kR, Resistor_SMD:R_0402_1005Metric, symbol Device:R
- removed R11, R18: 100kR, Resistor_SMD:R_0402_1005Metric, symbol Device:R
- removed R12, R13, R14, R15, R31: 47kR, Resistor_SMD:R_0402_1005Metric, symbol Device:R
- removed R16, R17: 1kR, Resistor_SMD:R_0402_1005Metric, symbol Device:R
- removed R25, R26, R27, R28: 0.15R, Resistor_SMD:R_0402_1005Metric, symbol Device:R
- removed R29, R9: 12kR, Resistor_SMD:R_0402_1005Metric, symbol Device:R
- removed R30: 2.2kR, Resistor_SMD:R_0402_1005Metric, symbol Device:R
- removed R32: 6.8kR, Resistor_SMD:R_0402_1005Metric, symbol Device:R
- removed R7, R8: 4.7kR, Resistor_SMD:R_0402_1005Metric, symbol Device:R
- removed S1: LCD Display ST7735S, Connector_JST:JST_SH_BM08B-SRSS-TB_1x08-1MP_P1.00mm_Vertical, symbol Connector_Generic:Conn_01x08
- removed SW1: TOP, Connector_JST:JST_SH_BM02B-SRSS-TB_1x02-1MP_P1.00mm_Vertical, symbol Switch:SW_Push
- removed SW2: BOTTOM, Connector_JST:JST_SH_BM02B-SRSS-TB_1x02-1MP_P1.00mm_Vertical, symbol Switch:SW_Push
- removed SW3: LEFT, Connector_JST:JST_SH_BM02B-SRSS-TB_1x02-1MP_P1.00mm_Vertical, symbol Switch:SW_Push
- removed SW4: RIGHT, Connector_JST:JST_SH_BM02B-SRSS-TB_1x02-1MP_P1.00mm_Vertical, symbol Switch:SW_Push
- removed SW5: SELECT, Connector_JST:JST_SH_BM02B-SRSS-TB_1x02-1MP_P1.00mm_Vertical, symbol Switch:SW_Push
- removed SW6: RETURN, Connector_JST:JST_SH_BM02B-SRSS-TB_1x02-1MP_P1.00mm_Vertical, symbol Switch:SW_Push
- removed SW7: RESET, Connector_JST:JST_SH_BM02B-SRSS-TB_1x02-1MP_P1.00mm_Vertical, symbol Switch:SW_Push
- removed U1: MCP23017x-x-ML, Package_DFN_QFN:QFN-28-1EP_6x6mm_P0.65mm_EP4.25x4.25mm, symbol Interface_Expansion:MCP23017x-x-ML
- removed U2: USB2512B_M2, ASTRAfootprints:QFN37P50_600X600X100L62X24T370N, symbol USB2512B_M2:USB2512B_M2
- removed U3: CH340C, Package_SO:SOIC-16_3.9x9.9mm_P1.27mm, symbol Interface_USB:CH340C
- removed U4: SPX3819M5-L-3-3, Package_TO_SOT_SMD:SOT-23-5, symbol Regulator_Linear:SPX3819M5-L-3-3
- removed U5: ESP32-WROOM-32UE, RF_Module:ESP32-WROOM-32UE, symbol RF_Module:ESP32-WROOM-32UE
- removed U6: AP62300WU, Package_TO_SOT_SMD:TSOT-23-6, symbol Regulator_Switching:AP62300WU
- removed U7, U8: TMC2209-LA, Package_DFN_QFN:VQFN-28-1EP_5x5mm_P0.5mm_EP3.7x3.7mm_ThermalVias, symbol Driver_Motor:TMC2209-LA
- removed Y1: Crystal_GND24, symbol Device:Crystal_GND24
Other:
- added sheet IMU & Expansion (imu.kicad_sch)
- added sheet MCU (mcu.kicad_sch)
- added sheet Motors (motors.kicad_sch)
- added sheet Power (power.kicad_sch)
- added sheet USB & Serial (usb.kicad_sch)
- added sheet User Interface (ui.kicad_sch)
- note added: "ASTRA Telescope Node - controller board, rev 7 Power: 12V in, protection, 5V + 3.3V bucks MCU: ESP32-WROOM-32UE USB & Serial: USB2512B hub (Pi Zero 2 host), CH340C, ESD, camera port Motors: 2x TMC2209 on one shared UART User Interface: MCP23017 buttons/LEDs, ST7735S LCD IMU & Expansion: BNO085 cable connector, 2x Qwiic Nets that cross sheets use global labels; power rails use power symbols."
- note added: "J5 BNO085 cable, J3/J4 Qwiic, IMU reset/INT pull-ups"
- note added: "P1 12V in, F1 PTC, Q1/D6 polarity, D7 TVS, U6 5V buck, U9 3.3V buck"
- note added: "U1 MCP23017, SW1-SW6 buttons, D1-D5 LEDs, S1 ST7735S LCD"
- note added: "U2 USB2512B hub + Y1, U3 CH340C, Q2/Q3 auto-program, J6, U10/U11 ESD, F2"
- note added: "U5 ESP32-WROOM-32UE reset/boot, I2C pull-ups, pin map"
- note added: "U7/U8 TMC2209 (shared UART) J1/J2 motor connectors, ENN pull-ups"

Commit message: V0.7 pcb
Other:
- note added: "ASTRA Telescope Node - controller board, rev 7 Power: 12V in, protection, 5V + 3.3V bucks MCU: ESP32-WROOM-32UE USB & Serial: USB2512B hub (Pi Zero 2 host), CH340C, ESD, camera port Motors: 2x TMC2209 on one shared UART User Interface: MCP23017 buttons/LEDs, ST7735S LCD IMU & Expansion: J3, JST-SH 4p I2C cable to the IMU board Nets that cross sheets use global labels; power rails use power symbol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"
- note added: "J3: I2C cable to the IMU board (GND, 3V3, SDA, SCL)"
- note removed: "ASTRA Telescope Node - controller board, rev 7 Power: 12V in, protection, 5V + 3.3V bucks MCU: ESP32-WROOM-32UE USB & Serial: USB2512B hub (Pi Zero 2 host), CH340C, ESD, camera port Motors: 2x TMC2209 on one shared UART User Interface: MCP23017 buttons/LEDs, ST7735S LCD IMU & Expansion: BNO085 cable connector, 2x Qwiic Nets that cross sheets use global labels; power rails use power symbols."
- note removed: "J5 BNO085 cable, J3/J4 Qwiic, IMU reset/INT pull-ups"
Changed lines of the file:
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@@
 		)
 	)
-	(text "J5 BNO085 cable, J3/J4 Qwiic,\nIMU reset/INT pull-ups"
+	(text "J3: I2C cable to the IMU board\n(GND, 3V3, SDA, SCL)"
 		(exclude_from_sim no)
 		(at 192.54 98.81 0)
@@
 		)
 	)
-	(text "ASTRA Telescope Node - controller board, rev 7\nPower: 12V in, protection, 5V + 3.3V bucks      MCU: ESP32-WROOM-32UE\nUSB & Serial: USB2512B hub (Pi Zero 2 host), CH340C, ESD, camera port\nMotors: 2x TMC2209 on one shared UART           User Interface: MCP23017 buttons/LEDs, ST7735S LCD\nIMU & Expansion: BNO085 cable connector, 2x Qwiic\nNets that cross sheets use global labels; power rails use power symbols."
+	(text "ASTRA Telescope Node - controller board, rev 7\nPower: 12V in, protection, 5V + 3.3V bucks      MCU: ESP32-WROOM-32UE\nUSB & Serial: USB2512B hub (Pi Zero 2 host), CH340C, ESD, camera port\nMotors: 2x TMC2209 on one shared UART           User Interface: MCP23017 buttons/LEDs, ST7735S LCD\nIMU & Expansion: J3, JST-SH 4p I2C cable to the IMU board\nNets that cross sheets use global labels; power rails use power symbols."
 		(exclude_from_sim no)
 		(at 30 150 0)

Commit message: v0.8
Other:
- sheet USB & Serial renamed Pi Link
- sheet Pi Link: file usb.kicad_sch -> pi_link.kicad_sch
- note added: "ASTRA Telescope Node - controller board, v0.8 Power: 12V in, protection, 5V + 3.3V bucks MCU: ESP32-WROOM-32UE Pi Link: J7 1x10 header to the Pi Zero 2 (5V power, UART0, ESP32 reset/boot via Q2/Q3) Motors: 2x TMC2209 on one shared UART User Interface: MCP23017 buttons/LEDs, ST7735S LCD IMU & Expansion: J3, JST-SH 4p I2C cable to the IMU board Nets that cross sheets use global labels; power rails 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"
- note added: "J7 1x10 to the Pi Zero 2 (5V, GND, UART0, Q2/Q3 auto-program)"
- note removed: "ASTRA Telescope Node - controller board, rev 7 Power: 12V in, protection, 5V + 3.3V bucks MCU: ESP32-WROOM-32UE USB & Serial: USB2512B hub (Pi Zero 2 host), CH340C, ESD, camera port Motors: 2x TMC2209 on one shared UART User Interface: MCP23017 buttons/LEDs, ST7735S LCD IMU & Expansion: J3, JST-SH 4p I2C cable to the IMU board Nets that cross sheets use global labels; power rails use power symbol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"
- note removed: "U2 USB2512B hub + Y1, U3 CH340C, Q2/Q3 auto-program, J6, U10/U11 ESD, F2"
Changed lines of the file:
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@@
 	(title_block
 		(title "ASTRA Telescope Node")
-		(date "2026-10-13")
-		(rev "7")
+		(date "2026-10-15")
+		(rev "v0.8")
 		(comment 1 "Author: Alex Grant-Parra")
 	)
@@
 		)
 	)
-	(text "U2 USB2512B hub + Y1, U3 CH340C,\nQ2/Q3 auto-program, J6, U10/U11 ESD, F2"
+	(text "J7 1x10 to the Pi Zero 2 (5V, GND,\nUART0, Q2/Q3 auto-program)"
 		(exclude_from_sim no)
 		(at 192.54 43.81 0)
@@
 			(color 0 0 0 0.0000)
 		)
-		(property "Sheetname" "USB & Serial"
+		(property "Sheetname" "Pi Link"
 			(at 190 39.2884 0)
 			(show_name no)
@@
 			)
 		)
-		(property "Sheetfile" "usb.kicad_sch"
+		(property "Sheetfile" "pi_link.kicad_sch"
 			(at 190 71.0646 0)
 			(show_name no)
@@
 		)
 	)
-	(text "ASTRA Telescope Node - controller board, rev 7\nPower: 12V in, protection, 5V + 3.3V bucks      MCU: ESP32-WROOM-32UE\nUSB & Serial: USB2512B hub (Pi Zero 2 host), CH340C, ESD, camera port\nMotors: 2x TMC2209 on one shared UART           User Interface: MCP23017 buttons/LEDs, ST7735S LCD\nIMU & Expansion: J3, JST-SH 4p I2C cable to the IMU board\nNets that cross sheets use global labels; power rails use power symbols."
+	(text "ASTRA Telescope Node - controller board, v0.8\nPower: 12V in, protection, 5V + 3.3V bucks      MCU: ESP32-WROOM-32UE\nPi Link: J7 1x10 header to the Pi Zero 2 (5V power, UART0, ESP32 reset/boot via Q2/Q3)\nMotors: 2x TMC2209 on one shared UART           User Interface: MCP23017 buttons/LEDs, ST7735S LCD\nIMU & Expansion: J3, JST-SH 4p I2C cable to the IMU board\nNets that cross sheets use global labels; power rails use power symbols."
 		(exclude_from_sim no)
 		(at 30 150 0)
