File: AstraController/ui.kicad_sch (KiCad schematic)
At the start: 22 parts, among them SW1 TOP, SW2 BOTTOM, SW3 LEFT, SW4 RIGHT, SW5 SELECT, SW6 RETURN, U1 MCP23017x-x-ML

Commit message: v0.8
Parts:
- C33: value 10uF -> 10uF 25V
- C6: value 100nF -> 100nF 50V
- R2: value 150R -> 330R
- R3, R4: value 47R -> 330R
Changed lines of the file:
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@@
 	(title_block
 		(title "ASTRA Telescope Node - User Interface")
-		(date "2026-10-13")
-		(rev "7")
+		(date "2026-10-15")
+		(rev "v0.8")
 		(comment 1 "Author: Alex Grant-Parra")
 	)
@@
 			)
 		)
-		(property "Value" "10uF"
+		(property "Value" "10uF 25V"
 			(at 39.624 58.42 0)
 			(show_name no)
@@
 			)
 		)
-		(property "Value" "47R"
+		(property "Value" "330R"
 			(at 72.136 96.774 90)
 			(show_name no)
@@
 			)
 		)
-		(property "Value" "150R"
+		(property "Value" "330R"
 			(at 72.136 94.234 90)
 			(show_name no)
@@
 			)
 		)
-		(property "Value" "47R"
+		(property "Value" "330R"
 			(at 72.136 99.314 90)
 			(show_name no)
@@
 			)
 		)
-		(property "Value" "100nF"
+		(property "Value" "100nF 50V"
 			(at 68.834 28.956 0)
 			(show_name no)
