File: AstraController/power.kicad_sch (KiCad schematic)
At the start: 27 parts, among them P1 12V-DC, Q1 AO3407A, U6 AP62300WU, U9 AP62300WU

Commit message: v0.8
Parts:
- C12, C16, C36, C40: value 100nF -> 100nF 50V
- C15: value 10uF -> 10uF 25V
- C35, C39: value 10uF 25V -> 10uF 50V
- C37, C38, C41, C42: value 22uF 10V -> 22uF 25V
- R29: value 52.3kR 1% -> 27kR 1%
- R30: value 10kR 1% -> 5.1kR 1%
- R33: value 31.6kR 1% -> 47kR 1%
- R34: value 10kR 1% -> 15kR 1%
Changed lines of the file:
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@@
 	(title_block
 		(title "ASTRA Telescope Node - Power")
-		(date "2026-10-13")
-		(rev "7")
+		(date "2026-10-15")
+		(rev "v0.8")
 		(comment 1 "Author: Alex Grant-Parra")
 	)
@@
 			)
 		)
-		(property "Value" "10uF"
+		(property "Value" "10uF 25V"
 			(at 57.404 101.6 0)
 			(show_name no)
@@
 			)
 		)
-		(property "Value" "100nF"
+		(property "Value" "100nF 50V"
 			(at 51.054 101.346 0)
 			(show_name no)
@@
 			)
 		)
-		(property "Value" "22uF 10V"
+		(property "Value" "22uF 25V"
 			(at 64.516 24.638 90)
 			(show_name no)
@@
 			)
 		)
-		(property "Value" "100nF"
+		(property "Value" "100nF 50V"
 			(at 56.642 35.56 0)
 			(show_name no)
@@
 			)
 		)
-		(property "Value" "10kR 1%"
+		(property "Value" "5.1kR 1%"
 			(at 49.53 52.07 90)
 			(show_name no)
@@
 			)
 		)
-		(property "Value" "52.3kR 1%"
+		(property "Value" "27kR 1%"
 			(at 39.37 52.07 90)
 			(show_name no)
@@
 			)
 		)
-		(property "Value" "10uF 25V"
+		(property "Value" "10uF 50V"
 			(at 23.876 32.512 0)
 			(show_name no)
@@
 			)
 		)
-		(property "Value" "22uF 10V"
+		(property "Value" "22uF 25V"
 			(at 64.77 36.068 90)
 			(show_name no)
@@
 			)
 		)
-		(property "Value" "100nF"
+		(property "Value" "100nF 50V"
 			(at 28.194 103.886 0)
 			(show_name no)
@@
 			)
 		)
-		(property "Description" "3A buck, 3.3V rail (ESP32, hub, CH340, MCP23017, LCD, IMU)"
+		(property "Description" "3A buck, 3.3V rail (ESP32, MCP23017, LCD, IMU)"
 			(at 137.16 38.1 0)
 			(hide yes)
@@
 			)
 		)
-		(property "Value" "10uF 25V"
+		(property "Value" "10uF 50V"
 			(at 126.746 33.782 0)
 			(show_name no)
@@
 			)
 		)
-		(property "Value" "100nF"
+		(property "Value" "100nF 50V"
 			(at 159.512 36.83 0)
 			(show_name no)
@@
 			)
 		)
-		(property "Value" "22uF 10V"
+		(property "Value" "22uF 25V"
 			(at 167.64 37.338 90)
 			(show_name no)
@@
 			)
 		)
-		(property "Value" "22uF 10V"
+		(property "Value" "22uF 25V"
 			(at 167.386 25.908 90)
 			(show_name no)
@@
 			)
 		)
-		(property "Value" "31.6kR 1%"
+		(property "Value" "47kR 1%"
 			(at 142.24 53.34 90)
 			(show_name no)
@@
 			)
 		)
-		(property "Value" "10kR 1%"
+		(property "Value" "15kR 1%"
 			(at 152.4 53.34 90)
 			(show_name no)
@@
 		)
 	)
+	(symbol
+		(lib_id "power:+3.3V")
+		(at 109.22 93.98 0)
+		(unit 1)
+		(body_style 1)
+		(exclude_from_sim no)
+		(in_bom yes)
+		(on_board yes)
+		(in_pos_files yes)
+		(dnp no)
+		(fields_autoplaced yes)
+		(property "Reference" "#PWR161"
+			(at 109.22 97.79 0)
+			(hide yes)
+			(show_name no)
+			(do_not_autoplace no)
+			(effects
+				(font
+					(size 1.27 1.27)
+				)
+			)
+		)
+		(property "Value" "+3.3V"
+			(at 109.22 88.9 0)
+			(show_name no)
+			(do_not_autoplace no)
+			(effects
+				(font
+					(size 1.27 1.27)
+				)
+			)
+		)
+		(property "Footprint" ""
+			(at 109.22 93.98 0)
+			(hide yes)
+			(show_name no)
+			(do_not_autoplace no)
+			(effects
+				(font
+					(size 1.27 1.27)
+				)
+			)
+		)
+		(property "Datasheet" ""
+			(at 109.22 93.98 0)
+			(hide yes)
+			(show_name no)
+			(do_not_autoplace no)
+			(effects
+				(font
+					(size 1.27 1.27)
+				)
+			)
+		)
+		(property "Description" "Power symbol creates a global label with name \"+3.3V\""
+			(at 109.22 93.98 0)
+			(hide yes)
+			(show_name no)
+			(do_not_autoplace no)
+			(effects
+				(font
+					(size 1.27 1.27)
+				)
+			)
+		)
+		(pin "1"
+		)
+		(instances
+			(project "ASTRA"
+				(path "/b5ed9a09-c593-4f23-9cbf-a235c2c98de3/3dd04e5d-a088-4160-b2d1-6a5bf40fa372"
+					(reference "#PWR161")
+					(unit 1)
+				)
+			)
+		)
+	)
+	(symbol
+		(lib_id "power:PWR_FLAG")
+		(at 109.22 96.52 180)
+		(unit 1)
+		(body_style 1)
+		(exclude_from_sim no)
+		(in_bom no)
+		(on_board no)
+		(in_pos_files yes)
+		(dnp no)
+		(property "Reference" "#FLG5"
+			(at 113.03 92.71 0)
+			(hide yes)
+			(show_name no)
+			(do_not_autoplace no)
+			(effects
+				(font
+					(size 1.27 1.27)
+				)
+			)
+		)
+		(property "Value" "PWR_FLAG"
+			(at 113.03 92.71 0)
+			(show_name no)
+			(do_not_autoplace no)
+			(effects
+				(font
+					(size 1.27 1.27)
+				)
+			)
+		)
+		(property "Footprint" ""
+			(at 109.22 96.52 0)
+			(hide yes)
+			(show_name no)
+			(do_not_autoplace no)
+			(effects
+				(font
+					(size 1.27 1.27)
+				)
+			)
+		)
+		(property "Datasheet" ""
+			(at 109.22 96.52 0)
+			(hide yes)
+			(show_name no)
+			(do_not_autoplace no)
+			(effects
+				(font
+					(size 1.27 1.27)
+				)
+			)
+		)
+		(property "Description" "Special symbol for telling ERC where power comes to a net"
+			(at 109.22 96.52 0)
+			(hide yes)
+			(show_name no)
+			(do_not_autoplace no)
+			(effects
+				(font
+					(size 1.27 1.27)
+				)
+			)
+		)
+		(pin "1"
+		)
+		(instances
+			(project "ASTRA"
+				(path "/b5ed9a09-c593-4f23-9cbf-a235c2c98de3/3dd04e5d-a088-4160-b2d1-6a5bf40fa372"
+					(reference "#FLG5")
+					(unit 1)
+				)
+			)
+		)
+	)
+	(wire
+		(pts
+			(xy 109.22 93.98) (xy 109.22 96.52)
+		)
+		(stroke
+			(width 0)
+			(type default)
+		)
+	)

Commit message: v0.8.1
Parts:
- removed C39: 10uF 50V, Capacitor_SMD:C_1206_3216Metric, symbol Device:C
- removed C40: 100nF 50V, Capacitor_SMD:C_0402_1005Metric, symbol Device:C
- removed C41, C42: 22uF 25V, Capacitor_SMD:C_0805_2012Metric, symbol Device:C
- removed L3: 3.3uH, Inductor_SMD:L_Wuerth_WE-PD-Typ-M-Typ-S, symbol Device:L
- removed R31: 47kR, Resistor_SMD:R_0402_1005Metric, symbol Device:R
- removed R32: 6.8kR, Resistor_SMD:R_0402_1005Metric, symbol Device:R
- removed R33: 47kR 1%, Resistor_SMD:R_0402_1005Metric, symbol Device:R
- removed R34: 15kR 1%, Resistor_SMD:R_0402_1005Metric, symbol Device:R
- added C48, C49, C51: 22uF 25V, Capacitor_SMD:C_0805_2012Metric, symbol Device:C
- added C50: 10uF 25V, Capacitor_SMD:C_0805_2012Metric, symbol Device:C
- added C52: 1nF 50V, Capacitor_SMD:C_0402_1005Metric, symbol Device:C
- added C53: 100pF 50V, Capacitor_SMD:C_0402_1005Metric, symbol Device:C
- added C54: 100nF 50V, Capacitor_SMD:C_0402_1005Metric, symbol Device:C
- added D8: SS34, Diode_SMD:D_SMA, symbol Device:D_Schottky
- added R39: 330R, Resistor_SMD:R_0402_1005Metric, symbol Device:R
- C36: value 100nF 50V -> 10nF 50V
- L2: value 3.3uH -> 15uH; footprint Inductor_SMD:L_Wuerth_WE-PD-Typ-M-Typ-S -> Inductor_SMD:L_Changjiang_FXL0840; MPN 7447789003 -> (none)
- R29: value 27kR 1% -> 15kR 1%
- R30: value 5.1kR 1% -> 4.7kR 1%
- U6: value AP62300WU -> TPS5430DDAR; footprint Package_TO_SOT_SMD:TSOT-23-6 -> Package_SO:TI_SO-PowerPAD-8_ThermalVias; symbol Regulator_Switching:AP62300WU -> Regulator_Switching:TPS5430DDA
- U9: value AP62300WU -> AMS1117-3.3; footprint Package_TO_SOT_SMD:TSOT-23-6 -> Package_TO_SOT_SMD:SOT-223-3_TabPin2; symbol Regulator_Switching:AP62300WU -> Regulator_Linear:AMS1117-3.3
Connections:
- net +12V: now also C35.1, U6.7 (VIN); no longer C35.2, U6.3 (IN), U9.3 (IN)
- net +3.3V: now also U9.2 (VO), C51.1
- net +5V: now also U9.3 (VI), C48.1, C49.1, C50.1, C52.1
- net GND: now also C35.2, U6.6 (GND), U6.9 (GNDPAD), C48.2, C49.2, C50.2, C51.2, C53.2, D8.2 (A), R39.2; no longer C35.1, U6.1 (GND)
- net 5V_FB: now reaches R29.2, R30.1, U6.4 (VSENSE)
- net 5V_FB: now also C52.2, C53.1, C54.1
- net 5V_SW: now reaches C36.2
- net 5V_SW: now also L2.1, U6.8 (PH), D8.1 (K); no longer U6.6 (BST)
- net BUCK_EN: no longer names the net of U6.5 (EN)
- net BUCK_EN: no longer U9.5 (EN)
- new net: C54.2, R39.1
- new net: C36.1, U6.1 (BOOT)
- now unconnected: U6.2 (SW)
- no-connect marks 0 -> 1
Other:
- note added: "12V IN -> F1 3A PTC -> Q1 reverse-polarity PFET (D6 clamps Vgs) -> +12V D7 SMAJ15A TVS on +12V (15V standoff, clamps ~24V: under the TPS5430 36V max) U6 TPS5430: +12V -> +5V buck, 3A, 500kHz. R29/R30 15k/4.7k -> 5.12V. L2 15uH (FXL0840-150-M), D8 SS34 catch diode, C36 10nF boot All-ceramic output (C37 C38 C48 C49) -> compensation per TI datasheet Fig 7-11: C52 1nF across R29, C53 100pF and C54 10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"
- note removed: "12V IN -> F1 3A PTC -> Q1 reverse-polarity PFET (D6 clamps Vgs) -> +12V D7 SMAJ15A TVS on +12V (15V standoff: off at 14.4V charging, clamps below AP62300 20V max) U6: +12V -> +5V (R29/R30 52.3k/10k, L2 3.3uH) U9: +12V -> +3.3V (R33/R34 31.6k/10k, L3 3.3uH) BUCK_EN: R31/R32 divider shared by U6 and U9 -> both rails start at ~9.3V Layout: keep each buck input loop (C35/C39 -> IN -> GND) and SW node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"
- moved on the sheet: C35, C36, C37, C38, L2, R29, R30

Commit message: v0.8.2
Parts:
- Q1: value AO3407A -> AO3401A
Changed lines of the file:
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@@
 			)
 		)
-		(property "Value" "AO3407A"
+		(property "Value" "AO3401A"
 			(at 72.39 60.96 90)
 			(show_name no)
@@
 			)
 		)
-		(property "Datasheet" "https://www.aosmd.com/res/datasheets/AO3407A.pdf"
+		(property "Datasheet" "https://www.aosmd.com/res/datasheets/AO3401A.pdf"
 			(at 68.58 57.15 0)
 			(hide yes)
