File: AstraController/ASTRA.kicad_pcb (KiCad board)
At the start: 4 copper layers, 85 x 50 mm, 54 parts, among them J1 RJ45 (NEMA 17), J2 RJ45 (NEMA 17), J3 RJ45 (BNO085), J5 USB_A, P1 12V-DC, SW1 TOP, SW2 BOTTOM, SW3 LEFT, SW4 RIGHT, SW5 SELECT, SW6 RETURN, SW7 RESET, T1 TMC2209, T2 TMC2209, U1 MCP23017x-x-SP, U3 CH340C, U4 SPX3819M5-L-3-3, U5 ESP32-WROOM-32UE

Commit message: frame and pcb ver 5.5
Parts:
- removed B1: XL4016E1 Buck Converter, ASTRAfootprints:Double 1x02 screw connector
- removed C5, C8: 100nF, Capacitor_SMD:C_0402_1005Metric
- removed J5: USB_A, Connector_USB:USB_A_Connfly_DS1095
- removed REF** (x4): MountingHole_2.5mm, MountingHole:MountingHole_2.5mm
- removed T1, T2: TMC2209, ASTRAfootprints:TMC2209module
- added C19: 100nF, Capacitor_SMD:C_0402_1005Metric, F.Cu at (197.9, 58.8)
- added C20: 10nF, Capacitor_SMD:C_0402_1005Metric, F.Cu at (197.9, 60.8)
- added C21: 100nF, Capacitor_SMD:C_0402_1005Metric, F.Cu at (197.9, 62.8)
- added C22: 100nF, Capacitor_SMD:C_0402_1005Metric, F.Cu at (200.7, 49.0)
- added C23: 18pF, Capacitor_SMD:C_0402_1005Metric, F.Cu at (200.7, 51.0)
- added C24: 18pF, Capacitor_SMD:C_0402_1005Metric, F.Cu at (200.7, 52.9)
- added C25: 10uF, Capacitor_SMD:C_0805_2012Metric, F.Cu at (188.9, 73.8)
- added C26: 100nF, Capacitor_SMD:C_0402_1005Metric, F.Cu at (200.7, 54.9)
- added C27: 2.2uF, Capacitor_SMD:C_0402_1005Metric, F.Cu at (200.7, 56.9)
- added C28: 22nF, Capacitor_SMD:C_0402_1005Metric, F.Cu at (200.7, 58.8)
- added C29: 100nF, Capacitor_SMD:C_0402_1005Metric, F.Cu at (200.7, 60.8)
- added C30: 22nF, Capacitor_SMD:C_0402_1005Metric, F.Cu at (200.7, 62.8)
- added C31: 2.2uF, Capacitor_SMD:C_0402_1005Metric, F.Cu at (203.6, 49.0)
- added C32: 100nF, Capacitor_SMD:C_0402_1005Metric, F.Cu at (203.6, 51.0)
- added C33: 10uF, Capacitor_SMD:C_0805_2012Metric, F.Cu at (188.9, 76.8)
- added C34: 10uF, Capacitor_SMD:C_0805_2012Metric, F.Cu at (188.9, 79.8)
- added C35: 10uF, Capacitor_SMD:C_0402_1005Metric, F.Cu at (203.6, 52.9)
- added C36: 100nF, Capacitor_SMD:C_0402_1005Metric, F.Cu at (203.6, 54.9)
- added C37: 22uF, Capacitor_SMD:C_0805_2012Metric, F.Cu at (188.9, 82.8)
- added C38: 22uF, Capacitor_SMD:C_0805_2012Metric, F.Cu at (188.9, 85.8)
- added F1: Polyfuse, Fuse:Fuse_2920_7451Metric, F.Cu at (216.6, 94.1)
- added J4: Conn_01x04, Connector_JST:JST_SH_BM04B-SRSS-TB_1x04-1MP_P1.00mm_Vertical, F.Cu at (184.4, 118.9)
- added J6: USB_A_Stacked, Connector_USB:USB_A_CUI_UJ2-ADH-TH_Horizontal_Stacked, F.Cu at (89.0, 59.1)
- added L2: L_Ferrite, Inductor_SMD:L_Wuerth_WE-PD-Typ-M-Typ-S, F.Cu at (216.3, 79.8)
- added Q1: AO3401A, Package_TO_SOT_SMD:SOT-23, F.Cu at (223.5, 82.1)
- added Q2: 2N3904, Package_TO_SOT_THT:TO-92_Inline, F.Cu at (188.7, 90.6)
- added Q3: 2N3904, Package_TO_SOT_THT:TO-92_Inline, F.Cu at (188.7, 96.4)
- added R10: 10kR, Resistor_SMD:R_0402_1005Metric, F.Cu at (209.4, 55.0)
- added R11: 100kR, Resistor_SMD:R_0402_1005Metric, F.Cu at (209.4, 57.0)
- added R12: 47kR, Resistor_SMD:R_0402_1005Metric, F.Cu at (209.4, 58.9)
- added R13: 47kR, Resistor_SMD:R_0402_1005Metric, F.Cu at (212.3, 49.0)
- added R14: 47kR, Resistor_SMD:R_0402_1005Metric, F.Cu at (212.3, 51.0)
- added R15: 47kR, Resistor_SMD:R_0402_1005Metric, F.Cu at (212.3, 53.0)
- added R16: 1kR, Resistor_SMD:R_0402_1005Metric, F.Cu at (212.3, 55.0)
- added R17: 1kR, Resistor_SMD:R_0402_1005Metric, F.Cu at (212.3, 57.0)
- added R18: 100kR, Resistor_SMD:R_0402_1005Metric, F.Cu at (212.3, 58.9)
- added R19: 10kR, Resistor_SMD:R_0402_1005Metric, F.Cu at (215.2, 49.0)
- added R20: 10kR, Resistor_SMD:R_0402_1005Metric, F.Cu at (215.2, 51.0)
- added R21: 10kR, Resistor_SMD:R_0402_1005Metric, F.Cu at (215.2, 53.0)
- added R22: 10kR, Resistor_SMD:R_0402_1005Metric, F.Cu at (215.2, 55.0)
- added R23: 10kR, Resistor_SMD:R_0402_1005Metric, F.Cu at (215.2, 57.0)
- added R24: 10kR, Resistor_SMD:R_0402_1005Metric, F.Cu at (215.2, 58.9)
- added R25: 0.15R, Resistor_SMD:R_0402_1005Metric, F.Cu at (218.1, 49.0)
- added R26: 0.15R, Resistor_SMD:R_0402_1005Metric, F.Cu at (218.1, 51.0)
- added R27: 0.15R, Resistor_SMD:R_0402_1005Metric, F.Cu at (218.1, 53.0)
- added R28: 0.15R, Resistor_SMD:R_0402_1005Metric, F.Cu at (218.1, 55.0)
- added R29: 12kR, Resistor_SMD:R_0402_1005Metric, F.Cu at (218.1, 57.0)
- added R30: 2.2kR, Resistor_SMD:R_0402_1005Metric, F.Cu at (218.1, 58.9)
- added R9: 12kR, Resistor_SMD:R_0402_1005Metric, F.Cu at (209.4, 53.0)
- added U2: USB2512B_M2, ASTRAfootprints:QFN37P50_600X600X100L62X24T370N, F.Cu at (218.2, 67.8)
- added U6: AP62300WU, Package_TO_SOT_SMD:TSOT-23-6, F.Cu at (196.1, 96.8)
- added U7: TMC2209-LA, Package_DFN_QFN:VQFN-28-1EP_5x5mm_P0.5mm_EP3.7x3.7mm_ThermalVias, F.Cu at (197.6, 78.9)
- added U8: TMC2209-LA, Package_DFN_QFN:VQFN-28-1EP_5x5mm_P0.5mm_EP3.7x3.7mm_ThermalVias, F.Cu at (197.6, 86.2)
- added Y1: Crystal, Crystal:Crystal_SMD_3225-4Pin_3.2x2.5mm, F.Cu at (223.7, 77.6)
- C10: value 10nF -> 100nF
- C15: footprint Capacitor_SMD:C_0402_1005Metric -> Capacitor_SMD:C_0805_2012Metric
- C17: value 47uF -> 100nF; footprint Capacitor_SMD:C_1206_3216Metric -> Capacitor_SMD:C_0402_1005Metric
- C18: value 1uF -> 10nF
- C7: value 100nF -> 1uF
- J1, J2: value RJ45 (NEMA 17) -> Nema17; footprint Connector_RJ:RJ45_Amphenol_54602-x08_Horizontal -> Connector_JST:JST_XH_B4B-XH-A_1x04_P2.50mm_Vertical
- J3: value RJ45 (BNO085) -> Conn_01x04; footprint Connector_RJ:RJ45_Amphenol_54602-x08_Horizontal -> Connector_JST:JST_SH_BM04B-SRSS-TB_1x04-1MP_P1.00mm_Vertical
- P1: footprint TerminalBlock:TerminalBlock_Xinya_XY308-2.54-2P_1x02_P2.54mm_Horizontal -> Connector_JST:JST_VH_B2P-VH_1x02_P3.96mm_Vertical
- R1, R2, R3, R4, R5: value 330R -> 100R
- S1: footprint ASTRAfootprints:Quadruple 1x02 screw connector -> Connector_JST:JST_SH_BM08B-SRSS-TB_1x08-1MP_P1.00mm_Vertical
- SW1, SW2, SW3, SW4, SW5, SW6, SW7: footprint TerminalBlock:TerminalBlock_Xinya_XY308-2.54-2P_1x02_P2.54mm_Horizontal -> Connector_JST:JST_SH_BM02B-SRSS-TB_1x02-1MP_P1.00mm_Vertical
- U1: value MCP23017x-x-SP -> MCP23017x-x-ML; footprint Package_DIP:DIP-28_W7.62mm -> Package_DFN_QFN:QFN-28-1EP_6x6mm_P0.65mm_EP4.25x4.25mm
- moved D5 132.1 mm to (221.8, 61.7)
- moved D4 132.1 mm to (221.8, 58.6)
- moved D3 132.0 mm to (221.8, 55.6)
- moved D2 131.9 mm to (221.8, 52.6)
- moved D1 131.9 mm to (221.8, 49.5)
- moved R5 118.5 mm to (206.5, 57.0), turned to 0 degrees
- moved R4 118.1 mm to (206.5, 55.0), turned to 0 degrees
- moved R3 117.8 mm to (206.5, 53.0), turned to 0 degrees
- moved R2 117.4 mm to (206.5, 51.0), turned to 0 degrees
- moved R1 117.1 mm to (206.5, 49.0), turned to 0 degrees
- moved C1 108.1 mm to (197.1, 69.5)
- moved P1 104.4 mm to (204.6, 80.0)
- moved C16 101.9 mm to (197.9, 52.9)
- moved C10 101.1 mm to (195.0, 60.8), turned to 0 degrees
- moved U4 100.7 mm to (196.1, 92.2)
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Connections:
- C17 pad 1: +5V -> GND
- C17 pad 2: GND -> Net-(U2-CRFILT)
- C18 pad 1: +3.3V -> GND
- C18 pad 2: GND -> Net-(U2-CRFILT)
- C4 pad 1: +12V -> +3.3V
- C7 pad 2: Net-(U5-EN) -> /DTR
- J1 pad 1: Net-(T1-M1B) -> Net-(J1-Pin_1)
- J1 pad 2: Net-(T1-M1B) -> Net-(J1-Pin_2)
- J1 pad 3: Net-(T1-M1A) -> Net-(J1-Pin_3)
- J1 pad 4: Net-(T1-M1A) -> Net-(J1-Pin_4)
- J2 pad 1: Net-(T2-M1B) -> Net-(J2-Pin_1)
- J2 pad 2: Net-(T2-M1B) -> Net-(J2-Pin_2)
- J2 pad 3: Net-(T2-M1A) -> Net-(J2-Pin_3)
- J2 pad 4: Net-(T2-M1A) -> Net-(J2-Pin_4)
- J3 pad 2: /SCL -> +3.3V
- J3 pad 3: GND -> /SDA
- J3 pad 4: /SDA -> /SCL
- P1 pad 2: +12V -> Net-(F1-Pad2)
- R6 pad 1: Net-(U5-EN) -> /DTR
- SW7 pad 2: Net-(U5-EN) -> /DTR
- U1 pad 1: /RETURN -> /RIGHT
- U1 pad 10: GND -> unconnected-(U1-NC-Pad10)
- U1 pad 11: unconnected-(U1-NC-Pad11) -> GND
- U1 pad 12: /SCL -> GND
- U1 pad 13: /SDA -> GND
- U1 pad 14: unconnected-(U1-NC-Pad14) -> Net-(U1-~{RESET})
- U1 pad 15: GND -> unconnected-(U1-INTB-Pad15)
- U1 pad 16: GND -> unconnected-(U1-INTA-Pad16)
- U1 pad 17: GND -> /YELLOW
- U1 pad 18: unconnected-(U1-~{RESET}-Pad18) -> /BLUE
- U1 pad 2: /TOP -> /RED
- U1 pad 21: /YELLOW -> unconnected-(U1-GPA4-Pad21)
- U1 pad 22: /BLUE -> unconnected-(U1-GPA5-Pad22)
- U1 pad 24: unconnected-(U1-GPA3-Pad24) -> /SELECT
- U1 pad 25: unconnected-(U1-GPA4-Pad25) -> /RETURN
- U1 pad 26: unconnected-(U1-GPA5-Pad26) -> /TOP
- U1 pad 27: unconnected-(U1-GPA6-Pad27) -> /BOTTOM
- U1 pad 28: /SELECT -> /LEFT
- U1 pad 3: /BOTTOM -> /GREEN
- U1 pad 4: /LEFT -> /WHITE
- U1 pad 5: /RIGHT -> +3.3V
- U1 pad 6: /RED -> GND
- U1 pad 7: /GREEN -> unconnected-(U1-NC-Pad7)
- U1 pad 8: /WHITE -> /SCL
- U1 pad 9: +3.3V -> /SDA
- U3 pad 13: /DTR -> Net-(U3-~{DTR})
- U3 pad 14: /RTS -> Net-(U3-~{RTS})
- U3 pad 5: Net-(J5-D+) -> /downstream2 D+
- U3 pad 6: Net-(J5-D-) -> /downstream2 D-
- U5 pad 10: /2PDN -> /2TX
- U5 pad 11: /2UART -> /2RX
- U5 pad 25: /DTR -> /RTS
- U5 pad 3: Net-(U5-EN) -> /DTR
- U5 pad 30: /1PDN -> /1TX
- U5 pad 31: /1UART -> /1RX
Routing:
- net +3.3V: track 174.5 -> 0.00 mm, vias 1 -> 0
- net +5V: track 103.9 -> 0.00 mm
- net /1EN: track 94.7 -> 0.00 mm, vias 1 -> 0
- net /SCL: track 86.6 -> 0.00 mm
- net /SDA: track 80.9 -> 0.00 mm, vias 2 -> 0
- net GND: track 65.7 -> 0.00 mm, vias 5 -> 0
- net /1STEP: track 64.4 -> 0.00 mm, vias 1 -> 0
- net /1DIR: track 62.5 -> 0.00 mm, vias 1 -> 0
- net +12V: track 58.7 -> 0.00 mm
- net /1PDN: track 52.5 -> 0.00 mm, vias 1 -> 0
- net /1UART: track 52.0 -> 0.00 mm, vias 1 -> 0
- net /BLUE: track 50.8 -> 0.00 mm
- net /RED: track 44.9 -> 0.00 mm, vias 1 -> 0
- net /RETURN: track 43.7 -> 0.00 mm
- net /YELLOW: track 43.5 -> 0.00 mm
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- removed copper zone on In1.Cu, net GND
Other:
- board text removed: "ASTRA V0.2"
- board text removed: "Buck"

Commit message: temp commit
Parts:
- J1, J2: footprint Connector_JST:JST_XH_B4B-XH-A_1x04_P2.50mm_Vertical -> Connector_JST:JST_PH_B6B-PH-K_1x06_P2.00mm_Vertical
- moved F1 136.3 mm to (81.0, 81.0), turned to -90 degrees
- moved P1 125.9 mm to (79.0, 90.0)
- moved U7 96.2 mm to (101.5, 84.5), turned to 180 degrees
- moved U8 80.6 mm to (117.0, 84.5), turned to 180 degrees
- moved J1 74.0 mm to (98.0, 92.0)
- moved U1 66.6 mm to (144.6, 81.2)
- moved J2 62.4 mm to (113.5, 92.0)
- moved SW7 59.7 mm to (134.5, 50.5), turned to -90 degrees
- moved SW6 55.8 mm to (129.3, 92.8), turned to 180 degrees
- moved SW5 52.2 mm to (135.2, 92.8), turned to 180 degrees
- moved Q1 46.5 mm to (182.8, 59.7)
- moved L2 44.7 mm to (173.3, 67.6)
- moved U3 36.3 mm to (227.5, 120.5), turned to 90 degrees
- moved SW4 35.3 mm to (141.2, 92.8), turned to 180 degrees
- moved R29 34.7 mm to (184.7, 66.0)
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Routing:
- net Net-(J1-Pin_2): track 0.00 -> 11.2 mm
- net Net-(J2-Pin_2): track 0.00 -> 11.1 mm
- net Net-(J1-Pin_1): track 0.00 -> 6.29 mm
- net Net-(J2-Pin_1): track 0.00 -> 6.24 mm
- net Net-(J1-Pin_4): track 0.00 -> 6.02 mm
- net Net-(J2-Pin_4): track 0.00 -> 5.97 mm
- net Net-(J1-Pin_3): track 0.00 -> 5.05 mm
- net Net-(J2-Pin_3): track 0.00 -> 5.00 mm
- added copper zone on In1.Cu, net GND

Commit message: v0.7
Parts:
- removed C10: 100nF, Capacitor_SMD:C_0402_1005Metric
- removed C18, C20: 10nF, Capacitor_SMD:C_0402_1005Metric
- removed R17: 1kR, Resistor_SMD:R_0402_1005Metric
- removed R24: 10kR, Resistor_SMD:R_0402_1005Metric
- removed U4: SPX3819M5-L-3-3, Package_TO_SOT_SMD:SOT-23-5
- added C14: 100nF, Capacitor_SMD:C_0402_1005Metric, F.Cu at (113.0, 54.1)
- added C39: 10uF 25V, Capacitor_SMD:C_1206_3216Metric, F.Cu at (136.3, 82.5)
- added C40: 100nF, Capacitor_SMD:C_0402_1005Metric, F.Cu at (136.1, 77.3)
- added C41: 22uF 10V, Capacitor_SMD:C_0805_2012Metric, F.Cu at (126.4, 85.3)
- added C42: 22uF 10V, Capacitor_SMD:C_0805_2012Metric, F.Cu at (128.6, 85.3)
- added C43: 22uF 10V, Capacitor_SMD:C_0805_2012Metric, F.Cu at (158.1, 55.5)
- added C44: 100nF, Capacitor_SMD:C_0402_1005Metric, F.Cu at (115.5, 53.4)
- added C45: 100nF, Capacitor_SMD:C_0402_1005Metric, F.Cu at (106.8, 66.8)
- added C46: 4.7uF 10V, Capacitor_SMD:C_0603_1608Metric, F.Cu at (113.1, 64.5)
- added D6: BZT52C10, Diode_SMD:D_SOD-123, F.Cu at (98.1, 75.5)
- added D7: SMAJ15A, Diode_SMD:D_SMA, F.Cu at (81.0, 81.5)
- added F2: PTC 0.75A hold 6V+, Fuse:Fuse_1206_3216Metric, F.Cu at (98.8, 65.8)
- added H1: M2.5, MountingHole:MountingHole_2.7mm_M2.5, F.Cu at (80.0, 49.0)
- added H2: M2.5, MountingHole:MountingHole_2.7mm_M2.5, F.Cu at (158.0, 49.0)
- added H3: M2.5, MountingHole:MountingHole_2.7mm_M2.5, F.Cu at (80.0, 92.0)
- added H4: M2.5, MountingHole:MountingHole_2.7mm_M2.5, F.Cu at (158.0, 92.0)
- added J5: BNO085_ext, Connector_JST:JST_SH_BM09B-SRSS-TB_1x09-1MP_P1.00mm_Vertical, F.Cu at (142.4, 48.2)
- added L3: 3.3uH, Inductor_SMD:L_Wuerth_WE-PD-Typ-M-Typ-S, F.Cu at (129.6, 79.5)
- added R31: 47kR, Resistor_SMD:R_0402_1005Metric, F.Cu at (125.3, 68.9)
- added R32: 6.8kR, Resistor_SMD:R_0402_1005Metric, F.Cu at (125.3, 67.8)
- added R33: 31.6kR 1%, Resistor_SMD:R_0402_1005Metric, F.Cu at (140.6, 80.7)
- added R34: 10kR 1%, Resistor_SMD:R_0402_1005Metric, F.Cu at (139.5, 80.7)
- added R35: 10kR, Resistor_SMD:R_0402_1005Metric, F.Cu at (147.0, 73.6)
- added R36: 10kR, Resistor_SMD:R_0402_1005Metric, F.Cu at (139.3, 51.6)
- added R37: 10kR, Resistor_SMD:R_0402_1005Metric, F.Cu at (157.1, 63.9)
- added R38: 10kR, Resistor_SMD:R_0402_1005Metric, F.Cu at (142.1, 80.7)
- added TP1: +12V, TestPoint:TestPoint_Pad_D1.0mm, F.Cu at (78.2, 79.5)
- added TP10: GND, TestPoint:TestPoint_Pad_D1.0mm, F.Cu at (159.7, 70.5)
- added TP11: SCL, TestPoint:TestPoint_Pad_D1.0mm, F.Cu at (102.5, 47.7)
- added TP12: SDA, TestPoint:TestPoint_Pad_D1.0mm, F.Cu at (102.5, 50.1)
- added TP13: TMC_UART, TestPoint:TestPoint_Pad_D1.0mm, F.Cu at (99.1, 81.1)
- added TP2: +5V, TestPoint:TestPoint_Pad_D1.0mm, F.Cu at (79.1, 56.4)
- added TP3: +3.3V, TestPoint:TestPoint_Pad_D1.0mm, F.Cu at (159.9, 58.3)
- added TP4: GND, TestPoint:TestPoint_Pad_D1.0mm, F.Cu at (79.1, 58.9)
- added TP5: GND, TestPoint:TestPoint_Pad_D1.0mm, F.Cu at (78.2, 82.1)
- added TP6: ESP32EN, TestPoint:TestPoint_Pad_D1.0mm, F.Cu at (159.7, 60.5)
- added TP7: GPIO0, TestPoint:TestPoint_Pad_D1.0mm, F.Cu at (159.7, 63.0)
- added TP8: UART1, TestPoint:TestPoint_Pad_D1.0mm, F.Cu at (159.7, 65.5)
- added TP9: UART2, TestPoint:TestPoint_Pad_D1.0mm, F.Cu at (159.7, 68.0)
- added U10: USBLC6-2SC6, Package_TO_SOT_SMD:SOT-23-6, F.Cu at (106.6, 56.1)
- added U11: USBLC6-2SC6, Package_TO_SOT_SMD:SOT-23-6, F.Cu at (103.4, 68.5)
- added U9: AP62300WU, Package_TO_SOT_SMD:TSOT-23-6, F.Cu at (136.1, 79.5)
- C1: value 680uF -> 680uF 25V low-ESR
- C2, C32: value 100nF -> 100nF 50V
- C26, C29: value 100nF -> 100nF 25V
- C27, C31: value 2.2uF -> 2.2uF 16V; footprint Capacitor_SMD:C_0402_1005Metric -> Capacitor_SMD:C_0603_1608Metric
- C28, C30: value 22nF -> 22nF 50V
- C34: value 10uF -> 100nF; footprint Capacitor_SMD:C_0805_2012Metric -> Capacitor_SMD:C_0402_1005Metric
- C35: value 10uF -> 10uF 25V; footprint Capacitor_SMD:C_0402_1005Metric -> Capacitor_SMD:C_1206_3216Metric
- C37, C38: value 22uF -> 22uF 10V
- F1: value Polyfuse -> PTC 3A hold 16V+
- L2: value L_Ferrite -> 3.3uH
- Q1: value AO3401A -> AO3407A
- Q2, Q3: value 2N3904 -> MMBT3904; footprint Package_TO_SOT_THT:TO-92_Inline -> Package_TO_SOT_SMD:SOT-23
- R1, R5: value 100R -> 330R
- R2: value 100R -> 150R
- R25, R26, R27, R28: value 0.15R -> 0.15R 0.5W 1%; footprint Resistor_SMD:R_0402_1005Metric -> Resistor_SMD:R_1206_3216Metric
- R29: value 12kR -> 52.3kR 1%
- R3, R4: value 100R -> 47R
- R30: value 2.2kR -> 10kR 1%
- R9: value 12kR -> 12kR 1%
- Y1: value Crystal -> 24MHz
- moved R25 138.4 mm to (88.1, 88.2)
- moved R26 132.1 mm to (94.1, 88.2), turned to 180 degrees
- moved R27 122.8 mm to (103.5, 88.2)
- moved U3 120.1 mm to (123.5, 60.5)
- moved C2 118.2 mm to (86.5, 85.8), turned to 90 degrees
- moved R28 116.5 mm to (109.5, 88.2), turned to 180 degrees
- moved C3 114.8 mm to (86.9, 81.3), turned to 180 degrees
- moved Y1 114.6 mm to (105.0, 61.8), turned to 90 degrees
- moved C32 111.3 mm to (101.9, 85.8), turned to 90 degrees
- moved C26 110.6 mm to (95.5, 81.7)
- moved C27 110.6 mm to (93.7, 79.6)
- moved C28 110.3 mm to (94.8, 83.3), turned to 90 degrees
- moved U2 106.6 mm to (112.0, 59.5), turned to 90 degrees
- moved C12 105.0 mm to (94.8, 66.7)
- moved C31 102.9 mm to (109.1, 79.6)
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Connections:
- net /1DIR renamed 1DIR
- net /1EN renamed 1EN
- net /1STEP renamed 1STEP
- net /1TX renamed TMC_TX
- net /2DIR renamed 2DIR
- net /2EN renamed 2EN
- net /2STEP renamed 2STEP
- net /BL renamed BL
- net /BLUE renamed /User Interface/BLUE
- net /BOTTOM renamed /User Interface/BOTTOM
- net /DC renamed DC
- net /DTR renamed ESP32EN
- net /GREEN renamed /User Interface/GREEN
- net /LEFT renamed /User Interface/LEFT
- net /MOSI renamed MOSI
- net /RED renamed /User Interface/RED
- net /RETURN renamed /User Interface/RETURN
- net /RIGHT renamed /User Interface/RIGHT
- net /RTS renamed GPIO0
- net /SCK renamed SCK
- net /SCL renamed SCL
- net /SDA renamed SDA
- net /T1_DIAG renamed T1_DIAG
- net /T2_DIAG renamed T2_DIAG
- net /TOP renamed /User Interface/TOP
- net /UART1 renamed UART1
- net /UART2 renamed UART2
- net /WHITE renamed /User Interface/WHITE
- net /YELLOW renamed /User Interface/YELLOW
- net /downstream1 D+ renamed /USB & Serial/downstream1 D+
- net /downstream1 D- renamed /USB & Serial/downstream1 D-
- net /downstream2 D+ renamed /USB & Serial/downstream2 D+
- net /downstream2 D- renamed /USB & Serial/downstream2 D-
- net /upstream D+ renamed /USB & Serial/upstream D+
- net /upstream D- renamed /USB & Serial/upstream D-
- C23 pad 1: Net-(C23-Pad1) -> /USB & Serial/XTALOUT
- C23 pad 2: /XTALOUT -> GND
- C24 pad 1: /XTALIN -> /USB & Serial/XTALIN
- C24 pad 2: Net-(C24-Pad2) -> GND
- C34 pad 2: /RST -> IMU_RST
- C35 pad 1: +12V -> GND
- C35 pad 2: GND -> +12V
- C9 pad 1: Net-(U3-V3) -> +3.3V
- F1 pad 1: Net-(Q1-S) -> Net-(Q1-D)
- J1 pad 2: Net-(J1-Pin_2) -> unconnected-(J1-Pin_2-Pad2)
- J1 pad 5: (no net) -> unconnected-(J1-Pin_5-Pad5)
- J1 pad 6: (no net) -> Net-(J1-Pin_6)
- J2 pad 2: Net-(J2-Pin_2) -> unconnected-(J2-Pin_2-Pad2)
- J2 pad 5: (no net) -> unconnected-(J2-Pin_5-Pad5)
- J2 pad 6: (no net) -> Net-(J2-Pin_6)
- J6 pad 5: +5V -> /USB & Serial/VBUS_CAM
- Q1 pad 2: Net-(Q1-S) -> +12V
- Q1 pad 3: +12V -> Net-(Q1-D)
- Q2 pad 1: GND -> Net-(Q2-B)
- Q2 pad 2: Net-(Q2-B) -> /USB & Serial/DTR
- Q3 pad 1: GND -> Net-(Q3-B)
- Q3 pad 2: Net-(Q3-B) -> /USB & Serial/RTS
- R16 pad 1: /1RX -> TMC_UART
- R20 pad 1: /RST -> IMU_RST
- R22 pad 2: Net-(U3-~{DTR}) -> /USB & Serial/DTR
- R23 pad 2: Net-(U3-~{RTS}) -> /USB & Serial/RTS
- S1 pad 5: /RES -> RES
- SW5 pad 1: /SELECT -> /User Interface/SELECT
- U1 pad 16: unconnected-(U1-INTA-Pad16) -> EXP_INT
- U1 pad 19: unconnected-(U1-GPA2-Pad19) -> /User Interface/SELECT
- U1 pad 24: /SELECT -> unconnected-(U1-GPA7-Pad24)
- U2 pad 32: /XTALOUT -> /USB & Serial/XTALOUT
- U2 pad 33: /XTALIN -> /USB & Serial/XTALIN
- U3 pad 13: Net-(U3-~{DTR}) -> /USB & Serial/DTR
- U3 pad 14: Net-(U3-~{RTS}) -> /USB & Serial/RTS
- U3 pad 16: +5V -> +3.3V
- U3 pad 4: Net-(U3-V3) -> +3.3V
- U5 pad 10: /2TX -> IMU_INT
- U5 pad 11: /2RX -> IMU_RST
- U5 pad 24: /RES -> unconnected-(U5-IO2-Pad24)
- U5 pad 26: unconnected-(U5-IO4-Pad26) -> RES
- U5 pad 31: /1RX -> TMC_UART
- U5 pad 5: unconnected-(U5-SENSOR_VN-Pad5) -> EXP_INT
- U6 pad 5: +12V -> /Power/BUCK_EN
- U7 pad 1: Net-(J1-Pin_4) -> Net-(J1-Pin_6)
- U7 pad 14: /1RX -> TMC_UART
- U7 pad 21: Net-(J1-Pin_2) -> Net-(J1-Pin_3)
- U7 pad 26: Net-(J1-Pin_3) -> Net-(J1-Pin_4)
- U8 pad 1: Net-(J2-Pin_4) -> Net-(J2-Pin_6)
- U8 pad 14: /2RX -> TMC_UART
- U8 pad 21: Net-(J2-Pin_2) -> Net-(J2-Pin_3)
- U8 pad 26: Net-(J2-Pin_3) -> Net-(J2-Pin_4)
- Y1 pad 1: Net-(C24-Pad2) -> /USB & Serial/XTALIN
- Y1 pad 2: Net-(C23-Pad1) -> GND
- Y1 pad 3: (no net) -> /USB & Serial/XTALOUT
- Y1 pad 4: (no net) -> GND
Routing:
- net SCL: track 0.00 -> 85.4 mm, vias 0 -> 8
- net SDA: track 0.00 -> 81.4 mm, vias 0 -> 5
- net T1_DIAG: track 0.00 -> 68.9 mm, vias 0 -> 2
- net 1STEP: track 0.00 -> 62.8 mm, vias 0 -> 2
- net 2STEP: track 0.00 -> 59.8 mm, vias 0 -> 6
- net 1DIR: track 0.00 -> 59.5 mm, vias 0 -> 2
- net TMC_UART: track 0.00 -> 59.0 mm, vias 0 -> 4
- net 1EN: track 0.00 -> 58.3 mm, vias 0 -> 2
- net +12V: track 0.00 -> 55.6 mm, vias 0 -> 17
- net 2DIR: track 0.00 -> 54.8 mm, vias 0 -> 4
- net T2_DIAG: track 0.00 -> 53.9 mm, vias 0 -> 2
- net /USB & Serial/DTR: track 0.00 -> 53.3 mm, vias 0 -> 4
- net GND: track 0.00 -> 51.6 mm, vias 0 -> 108
- net 2EN: track 0.00 -> 50.7 mm, vias 0 -> 2
- net EXP_INT: track 0.00 -> 48.7 mm, vias 0 -> 2
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- added copper zone on In2.Cu, net +12V
- added copper zone on In2.Cu, net +3.3V
- added copper zone on In2.Cu, net +5V
Other:
- board text added: "12V"
- board text added: "12V+"
- board text added: "3V3"
- board text added: "5V"
- board text added: "B"
- board text added: "BOTTOM"
- board text added: "EN"
- board text added: "G"
- board text added: "GND"
- board text added: "IMU"
- board text added: "IO0"
- board text added: "LCD"
- board text added: "LEFT"
- board text added: "M1"
- board text added: "M2"
- board text added: "PI:1-4 CAM:5-8"
- board text added: "QWIIC"
- board text added: "R"
- board text added: "RETURN"
- board text added: "RIGHT"
- board text added: "RST"
- board text added: "RX"
- board text added: "SCL"
- board text added: "SDA"
- board text added: "SELECT"
- board text added: "SELENO.v0.7"
- board text added: "TOP"
- board text added: "TX"
- board text added: "UART"
- board text added: "W"
- board text added: "Y"

Commit message: V0.7 pcb
Parts:
- removed C34: 100nF, Capacitor_SMD:C_0402_1005Metric
- removed J4: Conn_01x04, Connector_JST:JST_SH_BM04B-SRSS-TB_1x04-1MP_P1.00mm_Vertical
- removed J5: BNO085_ext, Connector_JST:JST_SH_BM09B-SRSS-TB_1x09-1MP_P1.00mm_Vertical
- removed R20, R37: 10kR, Resistor_SMD:R_0402_1005Metric
Connections:
- U5 pad 10: IMU_INT -> unconnected-(U5-IO25-Pad10)
- U5 pad 11: IMU_RST -> unconnected-(U5-IO26-Pad11)
Routing:
- net IMU_RST: track 35.0 -> 0.00 mm, vias 4 -> 0
- net IMU_INT: track 26.8 -> 0.00 mm, vias 3 -> 0
- net DC: track 0.00 -> 20.4 mm, vias 0 -> 2
- net MOSI: track 0.00 -> 15.8 mm
- net SCL: track 85.4 -> 90.1 mm, vias 8 -> 7
- net UART2: track 48.1 -> 52.6 mm, vias 2 -> 3
- net TMC_UART: track 59.0 -> 61.6 mm
- net 1EN: track 58.3 -> 60.4 mm
- net +3.3V: track 40.6 -> 38.6 mm, vias 43 -> 39
- net GND: track 51.6 -> 49.6 mm, vias 108 -> 103
- net UART1: track 45.6 -> 47.3 mm
- net T2_DIAG: track 53.9 -> 55.0 mm
- net SDA: track 81.4 -> 82.2 mm
- net GPIO0: track 43.1 -> 43.7 mm, vias 5 -> 3
- net 2STEP: track 59.8 -> 60.3 mm, vias 6 -> 8
Other:
- board text removed: "QWIIC"

Commit message: v0.8
Parts:
- removed C13, C14, C17, C19, C21, C22, C44, C45, C9: 100nF, Capacitor_SMD:C_0402_1005Metric
- removed C23, C24: 18pF, Capacitor_SMD:C_0402_1005Metric
- removed C25: 10uF, Capacitor_SMD:C_0805_2012Metric
- removed C46: 4.7uF 10V, Capacitor_SMD:C_0603_1608Metric
- removed F2: PTC 0.75A hold 6V+, Fuse:Fuse_1206_3216Metric
- removed J6: USB_A_Stacked, Connector_USB:USB_A_CUI_UJ2-ADH-TH_Horizontal_Stacked
- removed R10: 10kR, Resistor_SMD:R_0402_1005Metric
- removed R11, R18: 100kR, Resistor_SMD:R_0402_1005Metric
- removed R12, R13, R14, R15: 47kR, Resistor_SMD:R_0402_1005Metric
- removed R9: 12kR 1%, Resistor_SMD:R_0402_1005Metric
- removed U10, U11: USBLC6-2SC6, Package_TO_SOT_SMD:SOT-23-6
- removed U2: USB2512B_M2, ASTRAfootprints:QFN37P50_600X600X100L62X24T370N
- removed U3: CH340C, Package_SO:SOIC-16_3.9x9.9mm_P1.27mm
- removed Y1: 24MHz, Crystal:Crystal_SMD_3225-4Pin_3.2x2.5mm
- added C47: 22uF 25V, Capacitor_SMD:C_0805_2012Metric, F.Cu at (98.4, 85.4)
- added J7: Pi link 1x10, Connector_PinHeader_2.54mm:PinHeader_1x10_P2.54mm_Vertical, F.Cu at (84.9, 47.7)
- added TP14: GND, TestPoint:TestPoint_Pad_D1.0mm, F.Cu at (131.5, 76.5)
- added TP15: +3.3V, TestPoint:TestPoint_Pad_D1.0mm, F.Cu at (134.1, 76.5)
- added TP16: UART1, TestPoint:TestPoint_Pad_D1.0mm, F.Cu at (136.7, 76.5)
- added TP17: UART2, TestPoint:TestPoint_Pad_D1.0mm, F.Cu at (139.3, 76.5)
- added TP18: ESP32EN, TestPoint:TestPoint_Pad_D1.0mm, F.Cu at (131.5, 79.5)
- added TP19: GPIO0, TestPoint:TestPoint_Pad_D1.0mm, F.Cu at (134.1, 79.5)
- added TP20: Pi Link/DTR, TestPoint:TestPoint_Pad_D1.0mm, F.Cu at (136.7, 79.5)
- added TP21: Pi Link/RTS, TestPoint:TestPoint_Pad_D1.0mm, F.Cu at (139.3, 79.5)
- added TP22: 1STEP, TestPoint:TestPoint_Pad_D1.0mm, F.Cu at (110.0, 72.3)
- added TP23: 1DIR, TestPoint:TestPoint_Pad_D1.0mm, F.Cu at (113.4, 72.3)
- added TP24: 1EN, TestPoint:TestPoint_Pad_D1.0mm, F.Cu at (116.8, 72.3)
- added TP25: T1_DIAG, TestPoint:TestPoint_Pad_D1.0mm, F.Cu at (120.2, 72.3)
- added TP26: TMC_UART, TestPoint:TestPoint_Pad_D1.0mm, F.Cu at (123.6, 72.3)
- added TP27: 2STEP, TestPoint:TestPoint_Pad_D1.0mm, F.Cu at (110.0, 74.7)
- added TP28: 2DIR, TestPoint:TestPoint_Pad_D1.0mm, F.Cu at (113.4, 74.7)
- added TP29: 2EN, TestPoint:TestPoint_Pad_D1.0mm, F.Cu at (116.8, 74.7)
- added TP30: T2_DIAG, TestPoint:TestPoint_Pad_D1.0mm, F.Cu at (120.2, 74.7)
- added TP31: TMC_TX, TestPoint:TestPoint_Pad_D1.0mm, F.Cu at (143.8, 73.2)
- added TP32: Power/BUCK_EN, TestPoint:TestPoint_Pad_D1.0mm, F.Cu at (95.5, 64.0)
- added TP33: EXP_INT, TestPoint:TestPoint_Pad_D1.0mm, F.Cu at (138.1, 74.1)
- C11, C12, C16, C3, C36, C4, C40, C6: value 100nF -> 100nF 50V
- C15, C33: value 10uF -> 10uF 25V
- C26, C29: value 100nF 25V -> 100nF 50V
- C35, C39: value 10uF 25V -> 10uF 50V
- C37, C38, C41, C42, C43: value 22uF 10V -> 22uF 25V
- C7: value 1uF -> 1uF 25V
- R2: value 150R -> 330R
- R29: value 52.3kR 1% -> 27kR 1%
- R3, R4: value 47R -> 330R
- R30: value 10kR 1% -> 5.1kR 1%
- R33: value 31.6kR 1% -> 47kR 1%
- R34: value 10kR 1% -> 15kR 1%
- TP10: value GND -> MOSI
- TP11: value SCL -> DC
- TP12: value SDA -> RES
- TP13: value TMC_UART -> BL
- TP2: value +5V -> GND
- TP3: value +3.3V -> +5V
- TP5: value GND -> +3.3V
- TP6: value ESP32EN -> GND
- TP7: value GPIO0 -> SCL
- TP8: value UART1 -> SDA
- TP9: value UART2 -> SCK
- moved TP3 80.9 mm to (79.1, 56.4)
- moved TP7 51.2 mm to (110.8, 47.7)
- moved TP8 49.5 mm to (113.5, 47.7)
- moved TP5 44.2 mm to (118.1, 63.1)
- moved TP6 39.1 mm to (120.7, 63.1)
- moved TP10 38.5 mm to (123.5, 57.3)
- moved TP9 38.4 mm to (123.5, 55.1)
- moved C16 33.4 mm to (111.5, 62.8), turned to -90 degrees
- moved R31 32.8 mm to (92.9, 63.5)
- moved C15 32.6 mm to (109.7, 62.8), turned to -90 degrees
- moved R32 32.6 mm to (92.9, 64.6), turned to 180 degrees
- moved C39 31.2 mm to (114.7, 60.0)
- moved C41 31.2 mm to (104.8, 62.8)
- moved C40 31.2 mm to (114.5, 54.8)
- moved C42 31.2 mm to (107.0, 62.8)
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Connections:
- net /USB & Serial/DTR renamed /Pi Link/DTR
- net /USB & Serial/RTS renamed /Pi Link/RTS
- TP10 pad 1: GND -> MOSI
- TP11 pad 1: SCL -> DC
- TP12 pad 1: SDA -> RES
- TP13 pad 1: TMC_UART -> BL
- TP2 pad 1: +5V -> GND
- TP3 pad 1: +3.3V -> +5V
- TP5 pad 1: GND -> +3.3V
- TP6 pad 1: ESP32EN -> GND
- TP7 pad 1: GPIO0 -> SCL
- TP8 pad 1: UART1 -> SDA
- TP9 pad 1: UART2 -> SCK
Routing:
- net /USB & Serial/upstream D+: track 43.2 -> 0.00 mm, vias 1 -> 0
- net UART1: track 47.3 -> 86.4 mm, vias 2 -> 5
- net /USB & Serial/upstream D-: track 38.0 -> 0.00 mm, vias 1 -> 0
- net +12V: track 55.6 -> 20.1 mm, vias 17 -> 19
- net /USB & Serial/downstream1 D+: track 32.3 -> 0.00 mm
- net /USB & Serial/downstream1 D-: track 28.3 -> 0.00 mm
- net GPIO0: track 43.7 -> 18.1 mm, vias 3 -> 6
- net /USB & Serial/downstream2 D-: track 22.5 -> 0.00 mm
- net UART2: track 52.6 -> 73.2 mm, vias 3 -> 6
- net /USB & Serial/downstream2 D+: track 19.9 -> 0.00 mm
- net SCL: track 90.1 -> 76.2 mm, vias 7 -> 6
- net ESP32EN: track 43.8 -> 56.8 mm, vias 4 -> 5
- net +5V: track 21.1 -> 8.25 mm, vias 8 -> 7
- net /Pi Link/RTS: track 46.8 -> 57.5 mm, vias 4 -> 1
- net RES: track 26.6 -> 36.1 mm, vias 0 -> 5
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Other:
- board text added: "1DIAG"
- board text added: "1DIR"
- board text added: "1EN"
- board text added: "1STEP"
- board text added: "2DIAG"
- board text added: "2DIR"
- board text added: "2EN"
- board text added: "2STEP"
- board text added: "BEN"
- board text added: "BL"
- board text added: "DC"
- board text added: "DTR"
- board text added: "ESP32 PROG"
- board text added: "INT"
- board text added: "MOSI"
- board text added: "PI: EVEN ROW, PIN 2 ... PIN 20"
- board text added: "RES"
- board text added: "RTS"
- board text added: "SCK"
- board text added: "SELENO.v0.8"
- board text added: "TTX"
- board text removed: "PI:1-4 CAM:5-8"
- board text removed: "SELENO.v0.7"
