File: AstraController/ASTRA.kicad_pcb (KiCad board)
At the start: 4 copper layers, 85 x 50 mm, 123 parts, among them J1 Nema17, J2 Nema17, J3 Conn_01x04, J7 Pi link 1x10, P1 12V-DC, Q1 AO3407A, Q2 MMBT3904, Q3 MMBT3904, SW1 TOP, SW2 BOTTOM, SW3 LEFT, SW4 RIGHT, SW5 SELECT, SW6 RETURN, SW7 RESET, U1 MCP23017x-x-ML, U5 ESP32-WROOM-32UE, U6 AP62300WU, U7 TMC2209-LA, U8 TMC2209-LA, U9 AP62300WU

Commit message: v0.8.1
Parts:
- removed C39: 10uF 50V, Capacitor_SMD:C_1206_3216Metric
- removed C40: 100nF 50V, Capacitor_SMD:C_0402_1005Metric
- removed C41, C42: 22uF 25V, Capacitor_SMD:C_0805_2012Metric
- removed L3: 3.3uH, Inductor_SMD:L_Wuerth_WE-PD-Typ-M-Typ-S
- removed R31: 47kR, Resistor_SMD:R_0402_1005Metric
- removed R32: 6.8kR, Resistor_SMD:R_0402_1005Metric
- removed R33: 47kR 1%, Resistor_SMD:R_0402_1005Metric
- removed R34: 15kR 1%, Resistor_SMD:R_0402_1005Metric
- removed TP32: Power/BUCK_EN, TestPoint:TestPoint_Pad_D1.0mm
- added C48: 22uF 25V, Capacitor_SMD:C_0805_2012Metric, F.Cu at (87.9, 63.5)
- added C49: 22uF 25V, Capacitor_SMD:C_0805_2012Metric, F.Cu at (90.1, 63.5)
- added C50: 10uF 25V, Capacitor_SMD:C_0805_2012Metric, F.Cu at (102.9, 68.4)
- added C51: 22uF 25V, Capacitor_SMD:C_0805_2012Metric, F.Cu at (114.6, 66.1)
- added C52: 1nF 50V, Capacitor_SMD:C_0402_1005Metric, F.Cu at (90.5, 66.9)
- added C53: 100pF 50V, Capacitor_SMD:C_0402_1005Metric, F.Cu at (94.1, 66.9)
- added C54: 100nF 50V, Capacitor_SMD:C_0402_1005Metric, F.Cu at (95.3, 66.9)
- added D8: SS34, Diode_SMD:D_SMA, F.Cu at (99.0, 57.4)
- added R39: 330R, Resistor_SMD:R_0402_1005Metric, F.Cu at (96.5, 66.9)
- C36: value 100nF 50V -> 10nF 50V
- L2: value 3.3uH -> 15uH; footprint Inductor_SMD:L_Wuerth_WE-PD-Typ-M-Typ-S -> Inductor_SMD:L_Changjiang_FXL0840
- R29: value 27kR 1% -> 15kR 1%
- R30: value 5.1kR 1% -> 4.7kR 1%
- U6: value AP62300WU -> TPS5430DDAR; footprint Package_TO_SOT_SMD:TSOT-23-6 -> Package_SO:TI_SO-PowerPAD-8_ThermalVias
- U9: value AP62300WU -> AMS1117-3.3; footprint Package_TO_SOT_SMD:TSOT-23-6 -> Package_TO_SOT_SMD:SOT-223-3_TabPin2
- moved R29 12.0 mm to (91.7, 66.9)
- moved U9 10.6 mm to (109.1, 66.1)
- moved R30 10.6 mm to (92.9, 66.9)
- moved C35 8.10 mm to (103.4, 62.5), turned to -90 degrees
- moved C15 7.92 mm to (116.7, 66.5)
- moved C16 7.92 mm to (118.5, 66.5)
- moved U6 6.04 mm to (98.0, 62.5)
- moved C36 3.40 mm to (94.7, 58.1), turned to 90 degrees
- moved C37 2.40 mm to (83.5, 63.5)
- moved C38 2.40 mm to (85.7, 63.5)
Connections:
- net Net-(U6-FB) renamed /Power/5V_FB
- C35 pad 1: GND -> +12V
- C35 pad 2: +12V -> GND
- C36 pad 1: Net-(U6-SW) -> Net-(U6-BOOT)
- C36 pad 2: Net-(U6-BST) -> /Power/5V_SW
- L2 pad 1: Net-(U6-SW) -> /Power/5V_SW
- U6 pad 1: GND -> Net-(U6-BOOT)
- U6 pad 2: Net-(U6-SW) -> unconnected-(U6-NC-Pad2)
- U6 pad 3: +12V -> unconnected-(U6-NC-Pad3)
- U6 pad 5: /Power/BUCK_EN -> unconnected-(U6-EN-Pad5)
- U6 pad 6: Net-(U6-BST) -> GND
- U9 pad 2: Net-(U9-SW) -> +3.3V
- U9 pad 3: +12V -> +5V
Routing:
- net /Power/BUCK_EN: track 27.6 -> 0.00 mm, vias 2 -> 0
- net +5V: track 8.25 -> 31.2 mm, vias 7 -> 6
- net GND: track 44.9 -> 63.4 mm, vias 74 -> 70
- net /Power/5V_SW: track 0.00 -> 14.8 mm
- net Net-(U9-SW): track 5.93 -> 0.00 mm
- net Net-(U6-SW): track 5.93 -> 0.00 mm
- net +3.3V: track 30.7 -> 35.2 mm, vias 28 -> 26
- net Net-(U9-FB): track 3.47 -> 0.00 mm
- net /Power/5V_FB: track 3.47 -> 6.59 mm
- net Net-(U6-BOOT): track 0.00 -> 1.87 mm
- net +12V: track 20.1 -> 18.4 mm, vias 19 -> 18
- net Net-(U9-BST): track 1.51 -> 0.00 mm
- net Net-(U6-BST): track 1.51 -> 0.00 mm
- net Net-(C54-Pad2): track 0.00 -> 1.20 mm
- added copper zone on F.Cu, net +3.3V
Other:
- board text removed: "BEN"

Commit message: v0.8.2
Parts:
- Q1: value AO3407A -> AO3401A
Changed lines of the file:
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@@
 			)
 		)
-		(property "Value" "AO3407A"
+		(property "Value" "AO3401A"
 			(at 0 2.4 180)
 			(layer "F.Fab")
@@
 			)
 		)
-		(property "Datasheet" "https://www.aosmd.com/res/datasheets/AO3407A.pdf"
+		(property "Datasheet" "https://www.aosmd.com/res/datasheets/AO3401A.pdf"
 			(at 0 0 180)
 			(layer "F.Fab")

Commit message: v0.8.3
Parts:
- J1, J2: footprint Connector_JST:JST_PH_B6B-PH-K_1x06_P2.00mm_Vertical -> Connector_JST:JST_XH_B4B-XH-A_1x04_P2.50mm_Vertical
- moved J1 1.12 mm to (86.6, 91.5)
- moved J2 1.12 mm to (102.0, 91.5)
Connections:
- J1 pad 2: unconnected-(J1-Pin_2-Pad2) -> Net-(J1-Pin_2)
- J2 pad 2: unconnected-(J2-Pin_2-Pad2) -> Net-(J2-Pin_2)
- U7 pad 1: Net-(J1-Pin_6) -> Net-(J1-Pin_4)
- U7 pad 21: Net-(J1-Pin_3) -> Net-(J1-Pin_2)
- U7 pad 26: Net-(J1-Pin_4) -> Net-(J1-Pin_3)
- U8 pad 1: Net-(J2-Pin_6) -> Net-(J2-Pin_4)
- U8 pad 21: Net-(J2-Pin_3) -> Net-(J2-Pin_2)
- U8 pad 26: Net-(J2-Pin_4) -> Net-(J2-Pin_3)
Routing:
- net Net-(J2-Pin_6): track 9.67 -> 0.00 mm
- net Net-(J1-Pin_6): track 9.67 -> 0.00 mm
- net Net-(J1-Pin_2): track 0.00 -> 8.96 mm
- net Net-(J2-Pin_2): track 0.00 -> 8.96 mm
- net Net-(J1-Pin_3): track 9.67 -> 7.05 mm
- net Net-(J2-Pin_3): track 9.67 -> 7.05 mm
- net Net-(J2-Pin_1): track 12.6 -> 11.1 mm
- net Net-(J1-Pin_1): track 12.6 -> 11.1 mm
- net Net-(J2-Pin_4): track 7.55 -> 8.55 mm
- net Net-(J1-Pin_4): track 7.55 -> 8.55 mm
