File: AstraController/ASTRA.kicad_pcb (KiCad board)
At the start: 4 copper layers, 85 x 50 mm, 122 parts, among them J1 Nema17, J2 Nema17, J3 Conn_01x04, J7 Pi link 1x10, P1 12V-DC, Q1 AO3401A, Q2 MMBT3904, Q3 MMBT3904, SW1 TOP, SW2 BOTTOM, SW3 LEFT, SW4 RIGHT, SW5 SELECT, SW6 RETURN, SW7 RESET, U1 MCP23017x-x-ML, U5 ESP32-WROOM-32UE, U6 TPS5430DDAR, U7 TMC2209-LA, U8 TMC2209-LA, U9 AMS1117-3.3

Commit message: v0.8.4
Routing:
- net +5V: track 31.2 -> 35.6 mm, vias 6 -> 8
