File: AstraController/imu.kicad_sch (KiCad schematic)
At the start: 6 parts, among them J3 Conn_01x04, J4 Conn_01x04, J5 BNO085_ext

Commit message: V0.7 pcb
Parts:
- removed C34: 100nF, Capacitor_SMD:C_0402_1005Metric, symbol Device:C
- removed J4: Conn_01x04, Connector_JST:JST_SH_BM04B-SRSS-TB_1x04-1MP_P1.00mm_Vertical, symbol Connector_Generic:Conn_01x04
- removed J5: BNO085_ext, Connector_JST:JST_SH_BM09B-SRSS-TB_1x09-1MP_P1.00mm_Vertical, symbol Connector_Generic:Conn_01x09
- removed R20, R37: 10kR, Resistor_SMD:R_0402_1005Metric, symbol Device:R
Other:
- note added: "J3: I2C cable to the separate IMU board (1 GND, 2 3V3, 3 SDA, 4 SCL - Qwiic pinout). The IMU's own resistors and capacitors live on that board; bus pull-ups R7/R8 stay here."
- note removed: "AD0"
- note removed: "GND"
- note removed: "IMU_CS"
- note removed: "J5: cable to BNO085 breakout on the OTA dovetail (1:1 with its header). I2C address 0x4A (AD0=0), PS0=0 (I2C). Breakout PS1 must be low. J3/J4: Qwiic (GND, 3V3, SDA, SCL)."
- note removed: "PS0"
- note removed: "VCC"

Commit message: v0.8.3
Parts:
- J3: now left out of the parts list
Changed lines of the file:
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@@
 		(body_style 1)
 		(exclude_from_sim no)
-		(in_bom yes)
+		(in_bom no)
 		(on_board yes)
 		(in_pos_files yes)
