File: AstraController/motors.kicad_sch (KiCad schematic)
At the start: 22 parts, among them J1 Nema17, J2 Nema17, U7 TMC2209-LA, U8 TMC2209-LA

Commit message: v0.8
Parts:
- added C47: 22uF 25V, Capacitor_SMD:C_0805_2012Metric, symbol Device:C
- C26, C29: value 100nF 25V -> 100nF 50V
- C3, C4: value 100nF -> 100nF 50V
Connections:
- net +12V: now also C47.1
- net GND: now also C47.2
Other:
- note added: "Shared single-wire UART: R16 1k from ESP32 TX; U7 addr 0 (MS1=0), U8 addr 1 (MS1=1). Set microsteps over UART (U8 standalone would be 1/32). R35/R36 hold ENN high so drivers are OFF while the ESP32 boots. Rsense 0.15R 1206 0.5W -> 1.35A RMS max. J1/J2: coil A = pins 1-3, coil B = 4-6. Layout: thermal vias under U7/U8, short separate sense-resistor GND returns. C47 22uF 25V: extra VS ceramic betwe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"
- note removed: "Shared single-wire UART: R16 1k from ESP32 TX; U7 addr 0 (MS1=0), U8 addr 1 (MS1=1). Set microsteps over UART (U8 standalone would be 1/32). R35/R36 hold ENN high so drivers are OFF while the ESP32 boots. Rsense 0.15R 1206 0.5W -> 1.35A RMS max. J1/J2: coil A = pins 1-3, coil B = 4-6. Layout: thermal vias under U7/U8, short separate sense-resistor GND returns."

Commit message: v0.8.3
Parts:
- J1, J2: footprint Connector_JST:JST_PH_B6B-PH-K_1x06_P2.00mm_Vertical -> Connector_JST:JST_XH_B4B-XH-A_1x04_P2.50mm_Vertical; symbol Connector_Generic:Conn_01x06 -> Connector_Generic:Conn_01x04; now left out of the parts list
- R25, R26, R27, R28: now left out of the parts list
Connections:
- net at U7.1 (OB2): now also J1.4 (Pin_4); no longer J1.6 (Pin_6)
- net at U7.21 (OA2): now also J1.2 (Pin_2); no longer J1.3 (Pin_3)
- net at U7.26 (OB1): now also J1.3 (Pin_3); no longer J1.4 (Pin_4)
- net at J2.2 (Pin_2): now also U8.21 (OA2)
- net at J2.3 (Pin_3): now also U8.26 (OB1); no longer U8.21 (OA2)
- net at J2.4 (Pin_4): now also U8.1 (OB2); no longer U8.26 (OB1)
- no-connect marks 10 -> 6
Changed lines of the file:
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@@
 		(body_style 1)
 		(exclude_from_sim no)
-		(in_bom yes)
+		(in_bom no)
 		(on_board yes)
 		(in_pos_files yes)
@@
 	)
 	(symbol
-		(lib_id "Connector_Generic:Conn_01x06")
-		(at 83.82 53.34 0)
+		(lib_id "Connector_Generic:Conn_01x04")
+		(at 83.82 50.8 0)
 		(unit 1)
 		(body_style 1)
 		(exclude_from_sim no)
-		(in_bom yes)
+		(in_bom no)
 		(on_board yes)
 		(in_pos_files yes)
@@
 		(fields_autoplaced yes)
 		(property "Reference" "J1"
-			(at 86.36 53.3399 0)
+			(at 86.36 50.7999 0)
 			(show_name no)
 			(do_not_autoplace no)
@@
 		)
 		(property "Value" "Nema17"
-			(at 86.36 55.8799 0)
+			(at 86.36 53.3399 0)
 			(show_name no)
 			(do_not_autoplace no)
@@
 			)
 		)
-		(property "Footprint" "Connector_JST:JST_PH_B6B-PH-K_1x06_P2.00mm_Vertical"
-			(at 83.82 53.34 0)
+		(property "Footprint" "Connector_JST:JST_XH_B4B-XH-A_1x04_P2.50mm_Vertical"
+			(at 83.82 50.8 0)
 			(hide yes)
 			(show_name no)
@@
 		)
 		(property "Datasheet" ""
-			(at 83.82 53.34 0)
+			(at 83.82 50.8 0)
 			(hide yes)
 			(show_name no)
@@
 			)
 		)
-		(property "Description" "Stepper motor 1 (6-pin JST-PH, coil A = 1-3, coil B = 4-6)"
-			(at 83.82 53.34 0)
+		(property "Description" "Stepper motor 1 (4-pin JST-XH, coil A = 1-2, coil B = 3-4; standard PH2.0-6P to XH2.54-4P stepper cable)"
+			(at 83.82 50.8 0)
 			(hide yes)
 			(show_name no)
@@
 		(pin "4"
 		)
-		(pin "5"
-		)
-		(pin "6"
-		)
 		(pin "1"
 		)
@@
 		(body_style 1)
 		(exclude_from_sim no)
-		(in_bom yes)
+		(in_bom no)
 		(on_board yes)
 		(in_pos_files yes)
@@
 	(wire
 		(pts
-			(xy 73.66 50.8) (xy 76.2 50.8)
+			(xy 73.66 50.8) (xy 78.74 50.8)
 		)
 		(stroke
@@
 	(wire
 		(pts
-			(xy 76.2 50.8) (xy 76.2 53.34)
+			(xy 74.93 53.34) (xy 78.74 53.34)
 		)
 		(stroke
@@
 	(wire
 		(pts
-			(xy 76.2 53.34) (xy 78.74 53.34)
+			(xy 73.66 55.88) (xy 74.93 55.88)
 		)
 		(stroke
@@
 	(wire
 		(pts
-			(xy 73.66 55.88) (xy 78.74 55.88)
+			(xy 74.93 55.88) (xy 74.93 53.34)
 		)
 		(stroke
@@
 	(wire
 		(pts
-			(xy 76.2 58.42) (xy 76.2 60.96)
+			(xy 76.2 58.42) (xy 76.2 55.88)
 		)
 		(stroke
@@
 	(wire
 		(pts
-			(xy 76.2 60.96) (xy 78.74 60.96)
+			(xy 76.2 55.88) (xy 78.74 55.88)
 		)
 		(stroke
@@
 		)
 	)
-	(no_connect
-		(at 78.74 50.8)
-	)
-	(no_connect
-		(at 78.74 58.42)
-	)
 	(junction
 		(at 113.03 46.99)
@@
 		(body_style 1)
 		(exclude_from_sim no)
-		(in_bom yes)
+		(in_bom no)
 		(on_board yes)
 		(in_pos_files yes)
@@
 		(body_style 1)
 		(exclude_from_sim no)
-		(in_bom yes)
+		(in_bom no)
 		(on_board yes)
 		(in_pos_files yes)
@@
 	)
 	(symbol
-		(lib_id "Connector_Generic:Conn_01x06")
-		(at 83.82 119.38 0)
+		(lib_id "Connector_Generic:Conn_01x04")
+		(at 83.82 116.84 0)
 		(unit 1)
 		(body_style 1)
 		(exclude_from_sim no)
-		(in_bom yes)
+		(in_bom no)
 		(on_board yes)
 		(in_pos_files yes)
@@
 		(fields_autoplaced yes)
 		(property "Reference" "J2"
-			(at 86.36 119.3799 0)
+			(at 86.36 116.8399 0)
 			(show_name no)
 			(do_not_autoplace no)
@@
 		)
 		(property "Value" "Nema17"
-			(at 86.36 121.9199 0)
+			(at 86.36 119.3799 0)
 			(show_name no)
 			(do_not_autoplace no)
@@
 			)
 		)
-		(property "Footprint" "Connector_JST:JST_PH_B6B-PH-K_1x06_P2.00mm_Vertical"
-			(at 83.82 119.38 0)
+		(property "Footprint" "Connector_JST:JST_XH_B4B-XH-A_1x04_P2.50mm_Vertical"
+			(at 83.82 116.84 0)
 			(hide yes)
 			(show_name no)
@@
 		)
 		(property "Datasheet" ""
-			(at 83.82 119.38 0)
+			(at 83.82 116.84 0)
 			(hide yes)
 			(show_name no)
@@
 			)
 		)
-		(property "Description" "Stepper motor 2 (6-pin JST-PH, coil A = 1-3, coil B = 4-6)"
-			(at 83.82 119.38 0)
+		(property "Description" "Stepper motor 2 (4-pin JST-XH, coil A = 1-2, coil B = 3-4; standard PH2.0-6P to XH2.54-4P stepper cable)"
+			(at 83.82 116.84 0)
 			(hide yes)
 			(show_name no)
@@
 		(pin "3"
 		)
-		(pin "5"
-		)
 		(pin "4"
 		)
-		(pin "6"
-		)
 		(pin "1"
 		)
@@
 	(wire
 		(pts
-			(xy 73.66 116.84) (xy 76.2 116.84)
+			(xy 73.66 116.84) (xy 78.74 116.84)
 		)
 		(stroke
@@
 	(wire
 		(pts
-			(xy 76.2 116.84) (xy 76.2 119.38)
+			(xy 74.93 119.38) (xy 78.74 119.38)
 		)
 		(stroke
@@
 	(wire
 		(pts
-			(xy 76.2 119.38) (xy 78.74 119.38)
+			(xy 73.66 121.92) (xy 74.93 121.92)
 		)
 		(stroke
@@
 	(wire
 		(pts
-			(xy 73.66 121.92) (xy 78.74 121.92)
+			(xy 74.93 121.92) (xy 74.93 119.38)
 		)
 		(stroke
@@
 	(wire
 		(pts
-			(xy 76.2 124.46) (xy 76.2 127)
+			(xy 76.2 124.46) (xy 76.2 121.92)
 		)
 		(stroke
@@
 	(wire
 		(pts
-			(xy 76.2 127) (xy 78.74 127)
+			(xy 76.2 121.92) (xy 78.74 121.92)
 		)
 		(stroke
@@
 		)
 	)
-	(no_connect
-		(at 78.74 116.84)
-	)
-	(no_connect
-		(at 78.74 124.46)
-	)
 	(symbol
