File: AstraController/pi_link.kicad_sch (KiCad schematic)
At the start: 5 parts, among them J7 Pi link 1x10, Q2 MMBT3904, Q3 MMBT3904

Commit message: v0.8.3
Parts:
- J7: now left out of the parts list
Changed lines of the file:
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@@
 		(body_style 1)
 		(exclude_from_sim no)
-		(in_bom yes)
+		(in_bom no)
 		(on_board yes)
 		(in_pos_files yes)
