File: SelenoController/SELENO - Copy.kicad_sch (KiCad schematic)
At the start: 90 parts, among them J1 RJ45 (NEMA 17), J2 RJ45 (NEMA 17), J3 RJ45 (BNO085), J4 RJ45 (BNO085), J6 USB_A_Stacked, P1 12V-DC, Q1 AO3401A, Q2 2N3904, Q3 2N3904, SW1 TOP, SW2 BOTTOM, SW3 LEFT, SW4 RIGHT, SW5 SELECT, SW6 RETURN, SW7 RESET, U1 MCP23017x-x-SP, U2 USB2512B_M2, U3 CH340C, U4 SPX3819M5-L-3-3, U5 ESP32-WROOM-32UE, U7 TMC2209-LA, U8 TMC2209-LA, Y1 Crystal

Commit message: renames
Parts:
- B1: footprint ASTRAfootprints:Double 1x02 screw connector -> SELENOfootprints:Double 1x02 screw connector
- S1: footprint ASTRAfootprints:Quadruple 1x02 screw connector -> SELENOfootprints:Quadruple 1x02 screw connector
- U2: footprint ASTRAfootprints:QFN37P50_600X600X100L62X24T370N -> SELENOfootprints:QFN37P50_600X600X100L62X24T370N
Other:
- title: ASTRA Telescope Node -> SELENO Telescope Node
