File: SelenoController/SELENO.kicad_sch (KiCad schematic)
At the start: 0 parts

Commit message: renames
Other:
- note added: "SELENO Telescope Node - controller board, v0.8 Power: 12V in, protection, 5V + 3.3V bucks MCU: ESP32-WROOM-32UE Pi Link: J7 1x10 header to the Pi Zero 2 (5V power, UART0, ESP32 reset/boot via Q2/Q3) Motors: 2x TMC2209 on one shared UART User Interface: MCP23017 buttons/LEDs, ST7735S LCD IMU & Expansion: J3, JST-SH 4p I2C cable to the IMU board Nets that cross sheets use global labels; power rails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"
- note removed: "ASTRA Telescope Node - controller board, v0.8 Power: 12V in, protection, 5V + 3.3V bucks MCU: ESP32-WROOM-32UE Pi Link: J7 1x10 header to the Pi Zero 2 (5V power, UART0, ESP32 reset/boot via Q2/Q3) Motors: 2x TMC2209 on one shared UART User Interface: MCP23017 buttons/LEDs, ST7735S LCD IMU & Expansion: J3, JST-SH 4p I2C cable to the IMU board Nets that cross sheets use global labels; power rails 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"
- title: ASTRA Telescope Node -> SELENO Telescope Node
Changed lines of the file:
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@@
 	(paper "A4")
 	(title_block
-		(title "ASTRA Telescope Node")
+		(title "SELENO Telescope Node")
 		(date "2026-10-15")
 		(rev "v0.8")
@@
 		)
 		(instances
-			(project "ASTRA"
+			(project "SELENO"
 				(path "/b5ed9a09-c593-4f23-9cbf-a235c2c98de3"
 					(page "2")
@@
 		)
 		(instances
-			(project "ASTRA"
+			(project "SELENO"
 				(path "/b5ed9a09-c593-4f23-9cbf-a235c2c98de3"
 					(page "3")
@@
 		)
 		(instances
-			(project "ASTRA"
+			(project "SELENO"
 				(path "/b5ed9a09-c593-4f23-9cbf-a235c2c98de3"
 					(page "4")
@@
 		)
 		(instances
-			(project "ASTRA"
+			(project "SELENO"
 				(path "/b5ed9a09-c593-4f23-9cbf-a235c2c98de3"
 					(page "5")
@@
 		)
 		(instances
-			(project "ASTRA"
+			(project "SELENO"
 				(path "/b5ed9a09-c593-4f23-9cbf-a235c2c98de3"
 					(page "6")
@@
 		)
 		(instances
-			(project "ASTRA"
+			(project "SELENO"
 				(path "/b5ed9a09-c593-4f23-9cbf-a235c2c98de3"
 					(page "7")
@@
 		)
 	)
-	(text "ASTRA Telescope Node - controller board, v0.8\nPower: 12V in, protection, 5V + 3.3V bucks      MCU: ESP32-WROOM-32UE\nPi Link: J7 1x10 header to the Pi Zero 2 (5V power, UART0, ESP32 reset/boot via Q2/Q3)\nMotors: 2x TMC2209 on one shared UART           User Interface: MCP23017 buttons/LEDs, ST7735S LCD\nIMU & Expansion: J3, JST-SH 4p I2C cable to the IMU board\nNets that cross sheets use global labels; power rails use power symbols."
+	(text "SELENO Telescope Node - controller board, v0.8\nPower: 12V in, protection, 5V + 3.3V bucks      MCU: ESP32-WROOM-32UE\nPi Link: J7 1x10 header to the Pi Zero 2 (5V power, UART0, ESP32 reset/boot via Q2/Q3)\nMotors: 2x TMC2209 on one shared UART           User Interface: MCP23017 buttons/LEDs, ST7735S LCD\nIMU & Expansion: J3, JST-SH 4p I2C cable to the IMU board\nNets that cross sheets use global labels; power rails use power symbols."
 		(exclude_from_sim no)
 		(at 30 150 0)
