File: SelenoController/imu.kicad_sch (KiCad schematic)
At the start: 1 part, among them J3 Conn_01x04

Commit message: renames
Other:
- title: ASTRA Telescope Node - IMU & Expansion -> SELENO Telescope Node - IMU & Expansion
Changed lines of the file:
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@@
 	(paper "A4")
 	(title_block
-		(title "ASTRA Telescope Node - IMU & Expansion")
+		(title "SELENO Telescope Node - IMU & Expansion")
 		(date "2026-10-15")
 		(rev "v0.8")
@@
 		)
 		(instances
-			(project "ASTRA"
+			(project "SELENO"
 				(path "/b5ed9a09-c593-4f23-9cbf-a235c2c98de3/f761b0c1-fb2d-4800-881a-525f14ea580b"
 					(reference "#PWR047")
@@
 		)
 		(instances
-			(project "ASTRA"
+			(project "SELENO"
 				(path "/b5ed9a09-c593-4f23-9cbf-a235c2c98de3/f761b0c1-fb2d-4800-881a-525f14ea580b"
 					(reference "J3")
@@
 		)
 		(instances
-			(project "ASTRA"
+			(project "SELENO"
 				(path "/b5ed9a09-c593-4f23-9cbf-a235c2c98de3/f761b0c1-fb2d-4800-881a-525f14ea580b"
 					(reference "#PWR046")
