File: SelenoController/mcu.kicad_sch (KiCad schematic)
At the start: 8 parts, among them SW7 RESET, U5 ESP32-WROOM-32UE

Commit message: renames
Other:
- title: ASTRA Telescope Node - MCU -> SELENO Telescope Node - MCU
Changed lines of the file:
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@@
 	(paper "A4")
 	(title_block
-		(title "ASTRA Telescope Node - MCU")
+		(title "SELENO Telescope Node - MCU")
 		(date "2026-10-15")
 		(rev "v0.8")
@@
 		)
 		(instances
-			(project "ASTRA"
+			(project "SELENO"
 				(path "/b5ed9a09-c593-4f23-9cbf-a235c2c98de3/0f677968-202c-43df-9ca1-aea9a187cd34"
 					(reference "R7")
@@
 		)
 		(instances
-			(project "ASTRA"
+			(project "SELENO"
 				(path "/b5ed9a09-c593-4f23-9cbf-a235c2c98de3/0f677968-202c-43df-9ca1-aea9a187cd34"
 					(reference "#PWR09")
@@
 		)
 		(instances
-			(project "ASTRA"
+			(project "SELENO"
 				(path "/b5ed9a09-c593-4f23-9cbf-a235c2c98de3/0f677968-202c-43df-9ca1-aea9a187cd34"
 					(reference "#PWR049")
@@
 		)
 		(instances
-			(project "ASTRA"
+			(project "SELENO"
 				(path "/b5ed9a09-c593-4f23-9cbf-a235c2c98de3/0f677968-202c-43df-9ca1-aea9a187cd34"
 					(reference "#PWR07")
@@
 		)
 		(instances
-			(project "ASTRA"
+			(project "SELENO"
 				(path "/b5ed9a09-c593-4f23-9cbf-a235c2c98de3/0f677968-202c-43df-9ca1-aea9a187cd34"
 					(reference "#PWR08")
@@
 		)
 		(instances
-			(project "ASTRA"
+			(project "SELENO"
 				(path "/b5ed9a09-c593-4f23-9cbf-a235c2c98de3/0f677968-202c-43df-9ca1-aea9a187cd34"
 					(reference "R8")
@@
 		)
 		(instances
-			(project "ASTRA"
+			(project "SELENO"
 				(path "/b5ed9a09-c593-4f23-9cbf-a235c2c98de3/0f677968-202c-43df-9ca1-aea9a187cd34"
 					(reference "#PWR064")
@@
 		)
 		(instances
-			(project "ASTRA"
+			(project "SELENO"
 				(path "/b5ed9a09-c593-4f23-9cbf-a235c2c98de3/0f677968-202c-43df-9ca1-aea9a187cd34"
 					(reference "C7")
@@
 		)
 		(instances
-			(project "ASTRA"
+			(project "SELENO"
 				(path "/b5ed9a09-c593-4f23-9cbf-a235c2c98de3/0f677968-202c-43df-9ca1-aea9a187cd34"
 					(reference "SW7")
@@
 		)
 		(instances
-			(project "ASTRA"
+			(project "SELENO"
 				(path "/b5ed9a09-c593-4f23-9cbf-a235c2c98de3/0f677968-202c-43df-9ca1-aea9a187cd34"
 					(reference "U5")
@@
 		)
 		(instances
-			(project "ASTRA"
+			(project "SELENO"
 				(path "/b5ed9a09-c593-4f23-9cbf-a235c2c98de3/0f677968-202c-43df-9ca1-aea9a187cd34"
 					(reference "R6")
@@
 		)
 		(instances
-			(project "ASTRA"
+			(project "SELENO"
 				(path "/b5ed9a09-c593-4f23-9cbf-a235c2c98de3/0f677968-202c-43df-9ca1-aea9a187cd34"
 					(reference "#PWR065")
@@
 		)
 		(instances
-			(project "ASTRA"
+			(project "SELENO"
 				(path "/b5ed9a09-c593-4f23-9cbf-a235c2c98de3/0f677968-202c-43df-9ca1-aea9a187cd34"
 					(reference "#PWR034")
@@
 		)
 		(instances
-			(project "ASTRA"
+			(project "SELENO"
 				(path "/b5ed9a09-c593-4f23-9cbf-a235c2c98de3/0f677968-202c-43df-9ca1-aea9a187cd34"
 					(reference "C11")
@@
 		)
 		(instances
-			(project "ASTRA"
+			(project "SELENO"
 				(path "/b5ed9a09-c593-4f23-9cbf-a235c2c98de3/0f677968-202c-43df-9ca1-aea9a187cd34"
 					(reference "#PWR059")
@@
 		)
 		(instances
-			(project "ASTRA"
+			(project "SELENO"
 				(path "/b5ed9a09-c593-4f23-9cbf-a235c2c98de3/0f677968-202c-43df-9ca1-aea9a187cd34"
 					(reference "#PWR058")
@@
 		)
 		(instances
-			(project "ASTRA"
+			(project "SELENO"
 				(path "/b5ed9a09-c593-4f23-9cbf-a235c2c98de3/0f677968-202c-43df-9ca1-aea9a187cd34"
 					(reference "C43")
@@
 		)
 		(instances
-			(project "ASTRA"
+			(project "SELENO"
 				(path "/b5ed9a09-c593-4f23-9cbf-a235c2c98de3/0f677968-202c-43df-9ca1-aea9a187cd34"
 					(reference "#PWR135")
@@
 		)
 		(instances
-			(project "ASTRA"
+			(project "SELENO"
 				(path "/b5ed9a09-c593-4f23-9cbf-a235c2c98de3/0f677968-202c-43df-9ca1-aea9a187cd34"
 					(reference "#PWR136")
