File: SelenoController/motors.kicad_sch (KiCad schematic)
At the start: 23 parts, among them J1 Nema17, J2 Nema17, U7 TMC2209-LA, U8 TMC2209-LA

Commit message: renames
Other:
- title: ASTRA Telescope Node - Motors -> SELENO Telescope Node - Motors
