File: SelenoController/pi_link.kicad_sch (KiCad schematic)
At the start: 5 parts, among them J7 Pi link 1x10, Q2 MMBT3904, Q3 MMBT3904

Commit message: renames
Other:
- title: ASTRA Telescope Node - Pi Link -> SELENO Telescope Node - Pi Link
Changed lines of the file:
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@@
 	(paper "A4")
 	(title_block
-		(title "ASTRA Telescope Node - Pi Link")
+		(title "SELENO Telescope Node - Pi Link")
 		(date "2026-10-15")
 		(rev "v0.8")
@@
 		)
 		(instances
-			(project "ASTRA"
+			(project "SELENO"
 				(path "/b5ed9a09-c593-4f23-9cbf-a235c2c98de3/9ce2aa5b-7d28-44af-8b2e-b0a8b49da214"
 					(reference "Q3")
@@
 		)
 		(instances
-			(project "ASTRA"
+			(project "SELENO"
 				(path "/b5ed9a09-c593-4f23-9cbf-a235c2c98de3/9ce2aa5b-7d28-44af-8b2e-b0a8b49da214"
 					(reference "Q2")
@@
 		)
 		(instances
-			(project "ASTRA"
+			(project "SELENO"
 				(path "/b5ed9a09-c593-4f23-9cbf-a235c2c98de3/9ce2aa5b-7d28-44af-8b2e-b0a8b49da214"
 					(reference "R22")
@@
 		)
 		(instances
-			(project "ASTRA"
+			(project "SELENO"
 				(path "/b5ed9a09-c593-4f23-9cbf-a235c2c98de3/9ce2aa5b-7d28-44af-8b2e-b0a8b49da214"
 					(reference "R23")
@@
 		)
 		(instances
-			(project "ASTRA"
+			(project "SELENO"
 				(path "/b5ed9a09-c593-4f23-9cbf-a235c2c98de3/9ce2aa5b-7d28-44af-8b2e-b0a8b49da214"
 					(reference "J7")
@@
 		)
 		(instances
-			(project "ASTRA"
+			(project "SELENO"
 				(path "/b5ed9a09-c593-4f23-9cbf-a235c2c98de3/9ce2aa5b-7d28-44af-8b2e-b0a8b49da214"
 					(reference "#PWR156")
@@
 		)
 		(instances
-			(project "ASTRA"
+			(project "SELENO"
 				(path "/b5ed9a09-c593-4f23-9cbf-a235c2c98de3/9ce2aa5b-7d28-44af-8b2e-b0a8b49da214"
 					(reference "#PWR157")
@@
 		)
 		(instances
-			(project "ASTRA"
+			(project "SELENO"
 				(path "/b5ed9a09-c593-4f23-9cbf-a235c2c98de3/9ce2aa5b-7d28-44af-8b2e-b0a8b49da214"
 					(reference "#PWR158")
@@
 		)
 		(instances
-			(project "ASTRA"
+			(project "SELENO"
 				(path "/b5ed9a09-c593-4f23-9cbf-a235c2c98de3/9ce2aa5b-7d28-44af-8b2e-b0a8b49da214"
 					(reference "#PWR159")
@@
 		)
 		(instances
-			(project "ASTRA"
+			(project "SELENO"
 				(path "/b5ed9a09-c593-4f23-9cbf-a235c2c98de3/9ce2aa5b-7d28-44af-8b2e-b0a8b49da214"
 					(reference "#PWR160")
