File: SelenoController/power.kicad_sch (KiCad schematic)
At the start: 27 parts, among them P1 12V-DC, Q1 AO3401A, U6 TPS5430DDAR, U9 AMS1117-3.3

Commit message: renames
Other:
- title: ASTRA Telescope Node - Power -> SELENO Telescope Node - Power
