File: SelenoController/ui.kicad_sch (KiCad schematic)
At the start: 22 parts, among them SW1 TOP, SW2 BOTTOM, SW3 LEFT, SW4 RIGHT, SW5 SELECT, SW6 RETURN, U1 MCP23017x-x-ML

Commit message: renames
Other:
- title: ASTRA Telescope Node - User Interface -> SELENO Telescope Node - User Interface
Changed lines of the file:
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@@
 	(paper "A4")
 	(title_block
-		(title "ASTRA Telescope Node - User Interface")
+		(title "SELENO Telescope Node - User Interface")
 		(date "2026-10-15")
 		(rev "v0.8")
@@
 		)
 		(instances
-			(project "ASTRA"
+			(project "SELENO"
 				(path "/b5ed9a09-c593-4f23-9cbf-a235c2c98de3/eff2e076-62ae-4b3a-b069-f06b0977600a"
 					(reference "#PWR037")
@@
 		)
 		(instances
-			(project "ASTRA"
+			(project "SELENO"
 				(path "/b5ed9a09-c593-4f23-9cbf-a235c2c98de3/eff2e076-62ae-4b3a-b069-f06b0977600a"
 					(reference "U1")
@@
 		)
 		(instances
-			(project "ASTRA"
+			(project "SELENO"
 				(path "/b5ed9a09-c593-4f23-9cbf-a235c2c98de3/eff2e076-62ae-4b3a-b069-f06b0977600a"
 					(reference "R19")
@@
 		)
 		(instances
-			(project "ASTRA"
+			(project "SELENO"
 				(path "/b5ed9a09-c593-4f23-9cbf-a235c2c98de3/eff2e076-62ae-4b3a-b069-f06b0977600a"
 					(reference "#PWR021")
@@
 		)
 		(instances
-			(project "ASTRA"
+			(project "SELENO"
 				(path "/b5ed9a09-c593-4f23-9cbf-a235c2c98de3/eff2e076-62ae-4b3a-b069-f06b0977600a"
 					(reference "#PWR0107")
@@
 		)
 		(instances
-			(project "ASTRA"
+			(project "SELENO"
 				(path "/b5ed9a09-c593-4f23-9cbf-a235c2c98de3/eff2e076-62ae-4b3a-b069-f06b0977600a"
 					(reference "#PWR0106")
@@
 		)
 		(instances
-			(project "ASTRA"
+			(project "SELENO"
 				(path "/b5ed9a09-c593-4f23-9cbf-a235c2c98de3/eff2e076-62ae-4b3a-b069-f06b0977600a"
 					(reference "C33")
@@
 		)
 		(instances
-			(project "ASTRA"
+			(project "SELENO"
 				(path "/b5ed9a09-c593-4f23-9cbf-a235c2c98de3/eff2e076-62ae-4b3a-b069-f06b0977600a"
 					(reference "#PWR020")
@@
 		)
 		(instances
-			(project "ASTRA"
+			(project "SELENO"
 				(path "/b5ed9a09-c593-4f23-9cbf-a235c2c98de3/eff2e076-62ae-4b3a-b069-f06b0977600a"
 					(reference "#PWR031")
@@
 		)
 		(instances
-			(project "ASTRA"
+			(project "SELENO"
 				(path "/b5ed9a09-c593-4f23-9cbf-a235c2c98de3/eff2e076-62ae-4b3a-b069-f06b0977600a"
 					(reference "R3")
@@
 		)
 		(instances
-			(project "ASTRA"
+			(project "SELENO"
 				(path "/b5ed9a09-c593-4f23-9cbf-a235c2c98de3/eff2e076-62ae-4b3a-b069-f06b0977600a"
 					(reference "D4")
@@
 		)
 		(instances
-			(project "ASTRA"
+			(project "SELENO"
 				(path "/b5ed9a09-c593-4f23-9cbf-a235c2c98de3/eff2e076-62ae-4b3a-b069-f06b0977600a"
 					(reference "R1")
@@
 		)
 		(instances
-			(project "ASTRA"
+			(project "SELENO"
 				(path "/b5ed9a09-c593-4f23-9cbf-a235c2c98de3/eff2e076-62ae-4b3a-b069-f06b0977600a"
 					(reference "SW4")
@@
 		)
 		(instances
-			(project "ASTRA"
+			(project "SELENO"
 				(path "/b5ed9a09-c593-4f23-9cbf-a235c2c98de3/eff2e076-62ae-4b3a-b069-f06b0977600a"
 					(reference "R5")
@@
 		)
 		(instances
-			(project "ASTRA"
+			(project "SELENO"
 				(path "/b5ed9a09-c593-4f23-9cbf-a235c2c98de3/eff2e076-62ae-4b3a-b069-f06b0977600a"
 					(reference "SW1")
@@
 		)
 		(instances
-			(project "ASTRA"
+			(project "SELENO"
 				(path "/b5ed9a09-c593-4f23-9cbf-a235c2c98de3/eff2e076-62ae-4b3a-b069-f06b0977600a"
 					(reference "R2")
@@
 		)
 		(instances
-			(project "ASTRA"
+			(project "SELENO"
 				(path "/b5ed9a09-c593-4f23-9cbf-a235c2c98de3/eff2e076-62ae-4b3a-b069-f06b0977600a"
 					(reference "R4")
@@
 		)
 		(instances
-			(project "ASTRA"
+			(project "SELENO"
 				(path "/b5ed9a09-c593-4f23-9cbf-a235c2c98de3/eff2e076-62ae-4b3a-b069-f06b0977600a"
 					(reference "SW3")
@@
 		)
 		(instances
-			(project "ASTRA"
+			(project "SELENO"
 				(path "/b5ed9a09-c593-4f23-9cbf-a235c2c98de3/eff2e076-62ae-4b3a-b069-f06b0977600a"
 					(reference "SW6")
@@
 		)
 		(instances
-			(project "ASTRA"
+			(project "SELENO"
 				(path "/b5ed9a09-c593-4f23-9cbf-a235c2c98de3/eff2e076-62ae-4b3a-b069-f06b0977600a"
 					(reference "#PWR022")
@@
 		)
 		(instances
-			(project "ASTRA"
+			(project "SELENO"
 				(path "/b5ed9a09-c593-4f23-9cbf-a235c2c98de3/eff2e076-62ae-4b3a-b069-f06b0977600a"
 					(reference "D1")
@@
 		)
 		(instances
-			(project "ASTRA"
+			(project "SELENO"
 				(path "/b5ed9a09-c593-4f23-9cbf-a235c2c98de3/eff2e076-62ae-4b3a-b069-f06b0977600a"
 					(reference "SW2")
@@
 		)
 		(instances
-			(project "ASTRA"
+			(project "SELENO"
 				(path "/b5ed9a09-c593-4f23-9cbf-a235c2c98de3/eff2e076-62ae-4b3a-b069-f06b0977600a"
 					(reference "D2")
@@
 		)
 		(instances
-			(project "ASTRA"
+			(project "SELENO"
 				(path "/b5ed9a09-c593-4f23-9cbf-a235c2c98de3/eff2e076-62ae-4b3a-b069-f06b0977600a"
 					(reference "SW5")
@@
 		)
 		(instances
-			(project "ASTRA"
+			(project "SELENO"
 				(path "/b5ed9a09-c593-4f23-9cbf-a235c2c98de3/eff2e076-62ae-4b3a-b069-f06b0977600a"
 					(reference "D3")
@@
 		)
 		(instances
-			(project "ASTRA"
+			(project "SELENO"
 				(path "/b5ed9a09-c593-4f23-9cbf-a235c2c98de3/eff2e076-62ae-4b3a-b069-f06b0977600a"
 					(reference "D5")
@@
 		)
 		(instances
-			(project "ASTRA"
+			(project "SELENO"
 				(path "/b5ed9a09-c593-4f23-9cbf-a235c2c98de3/eff2e076-62ae-4b3a-b069-f06b0977600a"
 					(reference "S1")
@@
 		)
 		(instances
-			(project "ASTRA"
+			(project "SELENO"
 				(path "/b5ed9a09-c593-4f23-9cbf-a235c2c98de3/eff2e076-62ae-4b3a-b069-f06b0977600a"
 					(reference "#PWR025")
@@
 		)
 		(instances
-			(project "ASTRA"
+			(project "SELENO"
 				(path "/b5ed9a09-c593-4f23-9cbf-a235c2c98de3/eff2e076-62ae-4b3a-b069-f06b0977600a"
 					(reference "#PWR027")
@@
 		)
 		(instances
-			(project "ASTRA"
+			(project "SELENO"
 				(path "/b5ed9a09-c593-4f23-9cbf-a235c2c98de3/eff2e076-62ae-4b3a-b069-f06b0977600a"
 					(reference "#PWR023")
@@
 		)
 		(instances
-			(project "ASTRA"
+			(project "SELENO"
 				(path "/b5ed9a09-c593-4f23-9cbf-a235c2c98de3/eff2e076-62ae-4b3a-b069-f06b0977600a"
 					(reference "C6")
@@
 		)
 		(instances
-			(project "ASTRA"
+			(project "SELENO"
 				(path "/b5ed9a09-c593-4f23-9cbf-a235c2c98de3/eff2e076-62ae-4b3a-b069-f06b0977600a"
 					(reference "#PWR032")
@@
 		)
 		(instances
-			(project "ASTRA"
+			(project "SELENO"
 				(path "/b5ed9a09-c593-4f23-9cbf-a235c2c98de3/eff2e076-62ae-4b3a-b069-f06b0977600a"
 					(reference "#PWR033")
@@
 		)
 		(instances
-			(project "ASTRA"
+			(project "SELENO"
 				(path "/b5ed9a09-c593-4f23-9cbf-a235c2c98de3/eff2e076-62ae-4b3a-b069-f06b0977600a"
 					(reference "R38")
@@
 		)
 		(instances
-			(project "ASTRA"
+			(project "SELENO"
 				(path "/b5ed9a09-c593-4f23-9cbf-a235c2c98de3/eff2e076-62ae-4b3a-b069-f06b0977600a"
 					(reference "#PWR146")
